Commit message: Up to 26 on HW

File: body.urdf (robot description, URDF)
Before this commit: robot robot, 3 links, 2 joints
Joints:
- joint Torso_BackLeg: origin xyz=1 0 -1 rpy=0 0 0 -> xyz=1 0 1 rpy=0 0 0
- joint Torso_FrontLeg: origin xyz=-1 0 -1 rpy=0 0 0 -> xyz=2 0 1 rpy=0 0 0

Commit message: done

File: body.urdf (robot description, URDF)
Before this commit: robot robot, 3 links, 2 joints
Links:
- added link BackLowerLeg, mass 1; collision box size=0.2 0.2 1; visual box size=0.2 0.2 1
- added link FrontLowerLeg, mass 1; collision box size=0.2 0.2 1; visual box size=0.2 0.2 1
- added link LeftLeg, mass 1; collision box size=1 0.2 0.2; visual box size=1 0.2 0.2
- added link LeftLowerLeg, mass 1; collision box size=0.2 0.2 1; visual box size=0.2 0.2 1
- added link RightLeg, mass 1; collision box size=1 0.2 0.2; visual box size=1 0.2 0.2
- added link RightLowerLeg, mass 1; collision box size=0.2 0.2 1; visual box size=0.2 0.2 1
Joints:
- added joint Torso_BackLowerLeg: type revolute, parent BackLeg, child BackLowerLeg, origin xyz=0 -1 0 rpy=0 0 0, axis 1 0 0, limit lower=-3.14159 upper=3.14159 effort=0.0 velocity=0.0
- added joint Torso_FrontLowerLeg: type revolute, parent FrontLeg, child FrontLowerLeg, origin xyz=0 1 0 rpy=0 0 0, axis 1 0 0, limit lower=-3.14159 upper=3.14159 effort=0.0 velocity=0.0
- added joint Torso_LeftLeg: type revolute, parent Torso, child LeftLeg, origin xyz=-0.5 0 1 rpy=0 0 0, axis 0 1 0, limit lower=-3.14159 upper=3.14159 effort=0.0 velocity=0.0
- added joint Torso_LeftLowerLeg: type revolute, parent LeftLeg, child LeftLowerLeg, origin xyz=-1 0 0 rpy=0 0 0, axis 0 1 0, limit lower=-3.14159 upper=3.14159 effort=0.0 velocity=0.0
- added joint Torso_RightLeg: type revolute, parent Torso, child RightLeg, origin xyz=0.5 0 1 rpy=0 0 0, axis 0 1 0, limit lower=-3.14159 upper=3.14159 effort=0.0 velocity=0.0
- added joint Torso_RightLowerLeg: type revolute, parent RightLeg, child RightLowerLeg, origin xyz=1 0 0 rpy=0 0 0, axis 0 1 0, limit lower=-3.14159 upper=3.14159 effort=0.0 velocity=0.0

Commit message: milestone1 done

File: body.urdf (robot description, URDF)
Before this commit: robot robot, 9 links, 8 joints
Links:
- link BackLeg: geometry collision box size=0.5594459809617875 0.6608029676239529 0.39755752146891266; visual box size=0.5594459809617875 0.6608029676239529 0.39755752146891266
- link BackLowerLeg: geometry collision box size=0.31591663134601355 0.6861100903425529 1.7832503928155556; visual box size=0.31591663134601355 0.6861100903425529 1.7832503928155556
- link FrontLeg: geometry collision box size=0.3768606648025201 0.8757683825480878 0.6859586536164958; visual box size=0.3768606648025201 0.8757683825480878 0.6859586536164958
- link FrontLowerLeg: geometry collision box size=0.28243615964012186 0.7475279242020427 1.0639389490264282; visual box size=0.28243615964012186 0.7475279242020427 1.0639389490264282
- link LeftLeg: geometry collision box size=1.8376652294999525 0.6702151129670423 0.5923300850474513; visual box size=1.8376652294999525 0.6702151129670423 0.5923300850474513
- link LeftLowerLeg: geometry collision box size=0.49221471422068186 0.911189737298791 0.4770495148562377; visual box size=0.49221471422068186 0.911189737298791 0.4770495148562377
- link RightLeg: geometry collision box size=1.999122567253829 0.2900200121289124 0.7734287096766509; visual box size=1.999122567253829 0.2900200121289124 0.7734287096766509
- link RightLowerLeg: geometry collision box size=0.14651441325792125 0.4699821477255246 0.7807411912721441; visual box size=0.14651441325792125 0.4699821477255246 0.7807411912721441
Joints:
- joint Torso_BackLowerLeg: origin xyz=0 -1 0 rpy=0 0 0 -> xyz=0 -0.6608029676239529 0 rpy=0 0 0
- joint Torso_FrontLowerLeg: origin xyz=0 1 0 rpy=0 0 0 -> xyz=0 0.8757683825480878 0 rpy=0 0 0
- joint Torso_LeftLowerLeg: origin xyz=-1 0 0 rpy=0 0 0 -> xyz=-1.8376652294999525 0 0 rpy=0 0 0
- joint Torso_RightLowerLeg: origin xyz=1 0 0 rpy=0 0 0 -> xyz=1.999122567253829 0 0 rpy=0 0 0
