Commit message: m2 done

File: body8.urdf (robot description, URDF)
Before this commit: robot robot, 9 links, 8 joints
Links:
- link BackLeg: geometry collision box size=0.23675173169493685 2.0 0.36503357985236046; visual box size=0.23675173169493685 2.0 0.36503357985236046
- link BackLowerLeg: geometry collision box size=0.23423875940849934 0.30098677293179743 1.0209801641553342; visual box size=0.23423875940849934 0.30098677293179743 1.0209801641553342
- link FrontLeg: geometry collision box size=0.343707811096401 2.0 0.2548712878375734; visual box size=0.343707811096401 2.0 0.2548712878375734
- link FrontLowerLeg: geometry collision box size=0.1 0.34284744836990644 1.4684721415951694; visual box size=0.1 0.34284744836990644 1.4684721415951694
- link LeftLeg: geometry collision box size=2.0 0.31074557843639905 0.2088159821415129; visual box size=2.0 0.31074557843639905 0.2088159821415129
- link LeftLowerLeg: geometry collision box size=0.20055117314188348 0.24441150067611545 2.0; visual box size=0.20055117314188348 0.24441150067611545 2.0
- link RightLeg: geometry collision box size=2.0 0.1 0.1; visual box size=2.0 0.1 0.1
- link RightLowerLeg: geometry collision box size=0.3718738714206247 0.1412952769611191 2.0; visual box size=0.3718738714206247 0.1412952769611191 2.0
Joints:
- joint Torso_BackLeg: origin xyz=0 -0.5 1 rpy=0 0 0 -> xyz=0 -0.5 2.5 rpy=0 0 0
- joint Torso_BackLowerLeg: origin xyz=0 -0.6608029676239529 0 rpy=0 0 0 -> xyz=0 -2.0 0 rpy=0 0 0
- joint Torso_FrontLeg: origin xyz=0 0.5 1 rpy=0 0 0 -> xyz=0 0.5 2.5 rpy=0 0 0
- joint Torso_FrontLowerLeg: origin xyz=0 0.8757683825480878 0 rpy=0 0 0 -> xyz=0 2.0 0 rpy=0 0 0
- joint Torso_LeftLeg: origin xyz=-0.5 0 1 rpy=0 0 0 -> xyz=-0.5 0 2.5 rpy=0 0 0
- joint Torso_LeftLowerLeg: origin xyz=-1.8376652294999525 0 0 rpy=0 0 0 -> xyz=-2.0 0 0 rpy=0 0 0
- joint Torso_RightLeg: origin xyz=0.5 0 1 rpy=0 0 0 -> xyz=0.5 0 2.5 rpy=0 0 0
- joint Torso_RightLowerLeg: origin xyz=1.999122567253829 0 0 rpy=0 0 0 -> xyz=2.0 0 0 rpy=0 0 0
