Commit message: milestone 3 kinda

File: body5.urdf (robot description, URDF)
Before this commit: robot robot, 9 links, 8 joints
Links:
- link BackLeg: geometry collision box size=0.2324137712780591 2.0 0.1916561802312586; visual box size=0.2324137712780591 2.0 0.1916561802312586
- link BackLowerLeg: geometry collision box size=0.3191442515860623 0.1 0.9851838378874173; visual box size=0.3191442515860623 0.1 0.9851838378874173
- link FrontLeg: geometry collision box size=0.3455420600412598 1.8112404393374801 0.15337925425481533; visual box size=0.3455420600412598 1.8112404393374801 0.15337925425481533
- link FrontLowerLeg: geometry collision box size=0.10579788023908257 0.10667261216479838 1.336315091498813; visual box size=0.10579788023908257 0.10667261216479838 1.336315091498813
- link LeftLeg: geometry collision box size=2.0 0.1 0.20423892886219697; visual box size=2.0 0.1 0.20423892886219697
- link LeftLowerLeg: geometry collision box size=0.2857025112899702 0.2669989008808959 2.0; visual box size=0.2857025112899702 0.2669989008808959 2.0
- link RightLeg: geometry collision box size=2.0 0.1968680873044122 0.20298444559099896; visual box size=2.0 0.1968680873044122 0.20298444559099896
- link RightLowerLeg: geometry collision box size=0.1 0.1 2.0; visual box size=0.1 0.1 2.0
Joints:
- joint Torso_BackLowerLeg: origin xyz=0 -1.9746695689187843 0 rpy=0 0 0 -> xyz=0 -2.0 0 rpy=0 0 0
- joint Torso_FrontLowerLeg: origin xyz=0 2.0 0 rpy=0 0 0 -> xyz=0 1.8112404393374801 0 rpy=0 0 0
- joint Torso_LeftLowerLeg: origin xyz=-1.990996342904461 0 0 rpy=0 0 0 -> xyz=-2.0 0 0 rpy=0 0 0

File: body6.urdf (robot description, URDF)
Before this commit: robot robot, 9 links, 8 joints
Links:
- link BackLeg: geometry collision box size=0.3278924308348349 1.9847403739408427 0.1804960162231949; visual box size=0.3278924308348349 1.9847403739408427 0.1804960162231949
- link BackLowerLeg: geometry collision box size=0.31123652828778414 0.1825639780844548 0.8604811695129854; visual box size=0.31123652828778414 0.1825639780844548 0.8604811695129854
- link FrontLeg: geometry collision box size=0.2126603350867994 1.8678903326001313 0.1; visual box size=0.2126603350867994 1.8678903326001313 0.1
- link FrontLowerLeg: geometry collision box size=0.38014556757947154 0.3544376506330646 1.3243833305564796; visual box size=0.38014556757947154 0.3544376506330646 1.3243833305564796
- link LeftLeg: geometry collision box size=2.0 0.15149711219431916 0.3229322595246215; visual box size=2.0 0.15149711219431916 0.3229322595246215
- link LeftLowerLeg: geometry collision box size=0.1 0.1525946511604405 2.0; visual box size=0.1 0.1525946511604405 2.0
- link RightLeg: geometry collision box size=2.0 0.1 0.29846919832303725; visual box size=2.0 0.1 0.29846919832303725
- link RightLowerLeg: geometry collision box size=0.2462100805964895 0.23278536552102463 1.8831893815877352; visual box size=0.2462100805964895 0.23278536552102463 1.8831893815877352
Joints:
- joint Torso_BackLowerLeg: origin xyz=0 -2.0 0 rpy=0 0 0 -> xyz=0 -1.9847403739408427 0 rpy=0 0 0
- joint Torso_FrontLowerLeg: origin xyz=0 1.8448889396967072 0 rpy=0 0 0 -> xyz=0 1.8678903326001313 0 rpy=0 0 0
- joint Torso_LeftLowerLeg: origin xyz=-1.8684050711148505 0 0 rpy=0 0 0 -> xyz=-2.0 0 0 rpy=0 0 0

File: body7.urdf (robot description, URDF)
Before this commit: robot robot, 9 links, 8 joints
Links:
- link BackLeg: geometry collision box size=0.22555712928706728 2.0 0.26209442199922245; visual box size=0.22555712928706728 2.0 0.26209442199922245
- link BackLowerLeg: geometry collision box size=0.1 0.1 0.9498754590194132; visual box size=0.1 0.1 0.9498754590194132
- link FrontLeg: geometry collision box size=0.2723394673070961 1.9441500623484465 0.3562402211938481; visual box size=0.2723394673070961 1.9441500623484465 0.3562402211938481
- link FrontLowerLeg: geometry collision box size=0.1 0.2722138360126897 1.3618509490556303; visual box size=0.1 0.2722138360126897 1.3618509490556303
- link LeftLeg: geometry collision box size=1.9773494428061924 0.23511897519460476 0.1; visual box size=1.9773494428061924 0.23511897519460476 0.1
- link LeftLowerLeg: geometry collision box size=0.11313439848038476 0.19825537066281096 2.0; visual box size=0.11313439848038476 0.19825537066281096 2.0
- link RightLeg: geometry collision box size=1.807026586116077 0.1 0.1; visual box size=1.807026586116077 0.1 0.1
- link RightLowerLeg: geometry collision box size=0.11383797716580486 0.39586080692777914 1.809920819415227; visual box size=0.11383797716580486 0.39586080692777914 1.809920819415227
Joints:
- joint Torso_FrontLowerLeg: origin xyz=0 2.0 0 rpy=0 0 0 -> xyz=0 1.9441500623484465 0 rpy=0 0 0
- joint Torso_LeftLowerLeg: origin xyz=-1.9147555050317053 0 0 rpy=0 0 0 -> xyz=-1.9773494428061924 0 0 rpy=0 0 0
- joint Torso_RightLowerLeg: origin xyz=2.0 0 0 rpy=0 0 0 -> xyz=1.807026586116077 0 0 rpy=0 0 0

File: body8.urdf (robot description, URDF)
Before this commit: robot robot, 9 links, 8 joints
Links:
- link BackLeg: geometry collision box size=0.2671208519519055 2.0 0.1; visual box size=0.2671208519519055 2.0 0.1
- link BackLowerLeg: geometry collision box size=0.3455784693376207 0.2962365729117565 0.9156870444998051; visual box size=0.3455784693376207 0.2962365729117565 0.9156870444998051
- link FrontLeg: geometry collision box size=0.19010734680401536 2.0 0.3860648541992473; visual box size=0.19010734680401536 2.0 0.3860648541992473
- link FrontLowerLeg: geometry collision box size=0.33699585334097415 0.19808147978636004 1.4623628632676533; visual box size=0.33699585334097415 0.19808147978636004 1.4623628632676533
- link LeftLeg: geometry collision box size=1.9042011695558374 0.33810355661314123 0.3312038166408269; visual box size=1.9042011695558374 0.33810355661314123 0.3312038166408269
- link LeftLowerLeg: geometry collision box size=0.1 0.13624044034815297 2.0; visual box size=0.1 0.13624044034815297 2.0
- link RightLeg: geometry collision box size=1.9800159006181703 0.34135070371246734 0.3878271262633052; visual box size=1.9800159006181703 0.34135070371246734 0.3878271262633052
- link RightLowerLeg: geometry collision box size=0.1 0.220929374930031 1.9924745512853639; visual box size=0.1 0.220929374930031 1.9924745512853639
Joints:
- joint Torso_LeftLowerLeg: origin xyz=-2.0 0 0 rpy=0 0 0 -> xyz=-1.9042011695558374 0 0 rpy=0 0 0
- joint Torso_RightLowerLeg: origin xyz=2.0 0 0 rpy=0 0 0 -> xyz=1.9800159006181703 0 0 rpy=0 0 0

File: body9.urdf (robot description, URDF)
Before this commit: robot robot, 9 links, 8 joints
Links:
- link BackLeg: geometry collision box size=0.32302623343901393 1.982675326642601 0.1; visual box size=0.32302623343901393 1.982675326642601 0.1
- link BackLowerLeg: geometry collision box size=0.27235909778865036 0.3217177535147582 1.188820621279158; visual box size=0.27235909778865036 0.3217177535147582 1.188820621279158
- link FrontLeg: geometry collision box size=0.1 1.8382160637196594 0.23552248078175256; visual box size=0.1 1.8382160637196594 0.23552248078175256
- link FrontLowerLeg: geometry collision box size=0.1 0.17711372203587789 1.5562943699454548; visual box size=0.1 0.17711372203587789 1.5562943699454548
- link LeftLeg: geometry collision box size=1.859369333917983 0.1 0.1; visual box size=1.859369333917983 0.1 0.1
- link LeftLowerLeg: geometry collision box size=0.34151017034788567 0.23504409147452812 2.0; visual box size=0.34151017034788567 0.23504409147452812 2.0
- link RightLeg: geometry collision box size=1.9655968875843952 0.10460186942587382 0.17636862276596343; visual box size=1.9655968875843952 0.10460186942587382 0.17636862276596343
- link RightLowerLeg: geometry collision box size=0.3721551521944462 0.3398118494122844 2.0; visual box size=0.3721551521944462 0.3398118494122844 2.0
Joints:
- joint Torso_BackLowerLeg: origin xyz=0 -2.0 0 rpy=0 0 0 -> xyz=0 -1.982675326642601 0 rpy=0 0 0
- joint Torso_FrontLowerLeg: origin xyz=0 2.0 0 rpy=0 0 0 -> xyz=0 1.8382160637196594 0 rpy=0 0 0
- joint Torso_LeftLowerLeg: origin xyz=-1.9029732146247642 0 0 rpy=0 0 0 -> xyz=-1.859369333917983 0 0 rpy=0 0 0
- joint Torso_RightLowerLeg: origin xyz=1.8720823936861066 0 0 rpy=0 0 0 -> xyz=1.9655968875843952 0 0 rpy=0 0 0
