Commit message: symmetry added

File: body10.urdf (robot description, URDF)
Before this commit: robot robot, 9 links, 8 joints
Links:
- link BackLeg: geometry collision box size=0.1 1.8767691195714171 0.20968441200372767; visual box size=0.1 1.8767691195714171 0.20968441200372767
- link BackLowerLeg: geometry collision box size=0.3256123181511858 0.13734630039358806 1.0829536943020055; visual box size=0.3256123181511858 0.13734630039358806 1.0829536943020055
- link FrontLeg: geometry collision box size=0.1 1.8767691195714171 0.20968441200372767; visual box size=0.1 1.8767691195714171 0.20968441200372767
- link FrontLowerLeg: geometry collision box size=0.3256123181511858 0.13734630039358806 1.0829536943020055; visual box size=0.3256123181511858 0.13734630039358806 1.0829536943020055
- link LeftLeg: geometry collision box size=2.110298966186739 0.3646224329121472 0.1; visual box size=2.110298966186739 0.3646224329121472 0.1
- link LeftLowerLeg: geometry collision box size=0.3692739521474873 0.2849844751291148 0.8328213134631489; visual box size=0.3692739521474873 0.2849844751291148 0.8328213134631489
- link RightLeg: geometry collision box size=2.110298966186739 0.3646224329121472 0.1; visual box size=2.110298966186739 0.3646224329121472 0.1
- link RightLowerLeg: geometry collision box size=0.3692739521474873 0.2849844751291148 0.8328213134631489; visual box size=0.3692739521474873 0.2849844751291148 0.8328213134631489
Joints:
- joint Torso_BackLowerLeg: origin xyz=0 -2 0 rpy=0 0 0 -> xyz=0 -1.8767691195714171 0 rpy=0 0 0
- joint Torso_FrontLowerLeg: origin xyz=0 2 0 rpy=0 0 0 -> xyz=0 1.8767691195714171 0 rpy=0 0 0
- joint Torso_LeftLowerLeg: origin xyz=-2 0 0 rpy=0 0 0 -> xyz=-2.110298966186739 0 0 rpy=0 0 0
- joint Torso_RightLowerLeg: origin xyz=2 0 0 rpy=0 0 0 -> xyz=2.110298966186739 0 0 rpy=0 0 0

File: body11.urdf (robot description, URDF)
Before this commit: robot robot, 9 links, 8 joints
Links:
- link BackLeg: geometry collision box size=0.25185219705813716 1.9017698948772108 0.1; visual box size=0.25185219705813716 1.9017698948772108 0.1
- link BackLowerLeg: geometry collision box size=0.325527058068221 0.2758723584264712 0.940464968524241; visual box size=0.325527058068221 0.2758723584264712 0.940464968524241
- link FrontLeg: geometry collision box size=0.25185219705813716 1.9017698948772108 0.1; visual box size=0.25185219705813716 1.9017698948772108 0.1
- link FrontLowerLeg: geometry collision box size=0.325527058068221 0.2758723584264712 0.940464968524241; visual box size=0.325527058068221 0.2758723584264712 0.940464968524241
- link LeftLeg: geometry collision box size=2.111003577918722 0.3076150213338009 0.3146109479254682; visual box size=2.111003577918722 0.3076150213338009 0.3146109479254682
- link LeftLowerLeg: geometry collision box size=0.37074202498025877 0.25293268281417725 1.1566286275976938; visual box size=0.37074202498025877 0.25293268281417725 1.1566286275976938
- link RightLeg: geometry collision box size=2.111003577918722 0.3076150213338009 0.3146109479254682; visual box size=2.111003577918722 0.3076150213338009 0.3146109479254682
- link RightLowerLeg: geometry collision box size=0.37074202498025877 0.25293268281417725 1.1566286275976938; visual box size=0.37074202498025877 0.25293268281417725 1.1566286275976938
Joints:
- joint Torso_BackLowerLeg: origin xyz=0 -2 0 rpy=0 0 0 -> xyz=0 -1.9017698948772108 0 rpy=0 0 0
- joint Torso_FrontLowerLeg: origin xyz=0 2 0 rpy=0 0 0 -> xyz=0 1.9017698948772108 0 rpy=0 0 0
- joint Torso_LeftLowerLeg: origin xyz=-2 0 0 rpy=0 0 0 -> xyz=-2.111003577918722 0 0 rpy=0 0 0
- joint Torso_RightLowerLeg: origin xyz=2 0 0 rpy=0 0 0 -> xyz=2.111003577918722 0 0 rpy=0 0 0

File: body12.urdf (robot description, URDF)
Before this commit: robot robot, 9 links, 8 joints
Links:
- link BackLeg: geometry collision box size=0.506555943962548 1.8623866089559789 0.1; visual box size=0.506555943962548 1.8623866089559789 0.1
- link BackLowerLeg: geometry collision box size=0.1 0.14991337210127298 1.0495566091214872; visual box size=0.1 0.14991337210127298 1.0495566091214872
- link FrontLeg: geometry collision box size=0.506555943962548 1.8623866089559789 0.1; visual box size=0.506555943962548 1.8623866089559789 0.1
- link FrontLowerLeg: geometry collision box size=0.1 0.14991337210127298 1.0495566091214872; visual box size=0.1 0.14991337210127298 1.0495566091214872
- link LeftLeg: geometry collision box size=1.878309033324971 0.26418805438399784 0.45235994852662864; visual box size=1.878309033324971 0.26418805438399784 0.45235994852662864
- link LeftLowerLeg: geometry collision box size=0.4801149038726308 0.13650720289283397 1.154492833887685; visual box size=0.4801149038726308 0.13650720289283397 1.154492833887685
- link RightLeg: geometry collision box size=1.878309033324971 0.26418805438399784 0.45235994852662864; visual box size=1.878309033324971 0.26418805438399784 0.45235994852662864
- link RightLowerLeg: geometry collision box size=0.4801149038726308 0.13650720289283397 1.154492833887685; visual box size=0.4801149038726308 0.13650720289283397 1.154492833887685
Joints:
- joint Torso_BackLowerLeg: origin xyz=0 -2 0 rpy=0 0 0 -> xyz=0 -1.8623866089559789 0 rpy=0 0 0
- joint Torso_FrontLowerLeg: origin xyz=0 2 0 rpy=0 0 0 -> xyz=0 1.8623866089559789 0 rpy=0 0 0
- joint Torso_LeftLowerLeg: origin xyz=-2 0 0 rpy=0 0 0 -> xyz=-1.878309033324971 0 0 rpy=0 0 0
- joint Torso_RightLowerLeg: origin xyz=2 0 0 rpy=0 0 0 -> xyz=1.878309033324971 0 0 rpy=0 0 0

File: body13.urdf (robot description, URDF)
Before this commit: robot robot, 9 links, 8 joints
Links:
- link BackLeg: geometry collision box size=0.3673222707212471 2.026237450058545 0.1; visual box size=0.3673222707212471 2.026237450058545 0.1
- link BackLowerLeg: geometry collision box size=0.29241574184782476 0.35513842369729004 1.1673159640977266; visual box size=0.29241574184782476 0.35513842369729004 1.1673159640977266
- link FrontLeg: geometry collision box size=0.3673222707212471 2.026237450058545 0.1; visual box size=0.3673222707212471 2.026237450058545 0.1
- link FrontLowerLeg: geometry collision box size=0.29241574184782476 0.35513842369729004 1.1673159640977266; visual box size=0.29241574184782476 0.35513842369729004 1.1673159640977266
- link LeftLeg: geometry collision box size=2.0864836820466373 0.19327037407342873 0.14056674802120656; visual box size=2.0864836820466373 0.19327037407342873 0.14056674802120656
- link LeftLowerLeg: geometry collision box size=0.1544679572531058 0.31720487839569644 0.9228159186866225; visual box size=0.1544679572531058 0.31720487839569644 0.9228159186866225
- link RightLeg: geometry collision box size=2.0864836820466373 0.19327037407342873 0.14056674802120656; visual box size=2.0864836820466373 0.19327037407342873 0.14056674802120656
- link RightLowerLeg: geometry collision box size=0.1544679572531058 0.31720487839569644 0.9228159186866225; visual box size=0.1544679572531058 0.31720487839569644 0.9228159186866225
Joints:
- joint Torso_BackLowerLeg: origin xyz=0 -2 0 rpy=0 0 0 -> xyz=0 -2.026237450058545 0 rpy=0 0 0
- joint Torso_FrontLowerLeg: origin xyz=0 2 0 rpy=0 0 0 -> xyz=0 2.026237450058545 0 rpy=0 0 0
- joint Torso_LeftLowerLeg: origin xyz=-2 0 0 rpy=0 0 0 -> xyz=-2.0864836820466373 0 0 rpy=0 0 0
- joint Torso_RightLowerLeg: origin xyz=2 0 0 rpy=0 0 0 -> xyz=2.0864836820466373 0 0 rpy=0 0 0

File: body14.urdf (robot description, URDF)
Before this commit: robot robot, 9 links, 8 joints
Links:
- link BackLeg: geometry collision box size=0.3717452505195169 2.3112030941718085 0.2086140908152814; visual box size=0.3717452505195169 2.3112030941718085 0.2086140908152814
- link BackLowerLeg: geometry collision box size=0.4073806242471627 0.1 0.9388608465930692; visual box size=0.4073806242471627 0.1 0.9388608465930692
- link FrontLeg: geometry collision box size=0.3717452505195169 2.3112030941718085 0.2086140908152814; visual box size=0.3717452505195169 2.3112030941718085 0.2086140908152814
- link FrontLowerLeg: geometry collision box size=0.4073806242471627 0.1 0.9388608465930692; visual box size=0.4073806242471627 0.1 0.9388608465930692
- link LeftLeg: geometry collision box size=1.8940597804259327 0.10542245171237999 0.2530846748251961; visual box size=1.8940597804259327 0.10542245171237999 0.2530846748251961
- link LeftLowerLeg: geometry collision box size=0.1 0.461466829059783 1.0395184209068344; visual box size=0.1 0.461466829059783 1.0395184209068344
- link RightLeg: geometry collision box size=1.8940597804259327 0.10542245171237999 0.2530846748251961; visual box size=1.8940597804259327 0.10542245171237999 0.2530846748251961
- link RightLowerLeg: geometry collision box size=0.1 0.461466829059783 1.0395184209068344; visual box size=0.1 0.461466829059783 1.0395184209068344
Joints:
- joint Torso_BackLowerLeg: origin xyz=0 -2 0 rpy=0 0 0 -> xyz=0 -2.3112030941718085 0 rpy=0 0 0
- joint Torso_FrontLowerLeg: origin xyz=0 2 0 rpy=0 0 0 -> xyz=0 2.3112030941718085 0 rpy=0 0 0
- joint Torso_LeftLowerLeg: origin xyz=-2 0 0 rpy=0 0 0 -> xyz=-1.8940597804259327 0 0 rpy=0 0 0
- joint Torso_RightLowerLeg: origin xyz=2 0 0 rpy=0 0 0 -> xyz=1.8940597804259327 0 0 rpy=0 0 0

File: body15.urdf (robot description, URDF)
Before this commit: robot robot, 9 links, 8 joints
Links:
- link BackLeg: geometry collision box size=0.3519842122454529 1.908138372914677 0.1; visual box size=0.3519842122454529 1.908138372914677 0.1
- link BackLowerLeg: geometry collision box size=0.2092883038953388 0.23075226013422878 1.0001375365028238; visual box size=0.2092883038953388 0.23075226013422878 1.0001375365028238
- link FrontLeg: geometry collision box size=0.3519842122454529 1.908138372914677 0.1; visual box size=0.3519842122454529 1.908138372914677 0.1
- link FrontLowerLeg: geometry collision box size=0.2092883038953388 0.23075226013422878 1.0001375365028238; visual box size=0.2092883038953388 0.23075226013422878 1.0001375365028238
- link LeftLeg: geometry collision box size=1.8002263045399527 0.1 0.1; visual box size=1.8002263045399527 0.1 0.1
- link LeftLowerLeg: geometry collision box size=0.1 0.1 1.0734182771900216; visual box size=0.1 0.1 1.0734182771900216
- link RightLeg: geometry collision box size=1.8002263045399527 0.1 0.1; visual box size=1.8002263045399527 0.1 0.1
- link RightLowerLeg: geometry collision box size=0.1 0.1 1.0734182771900216; visual box size=0.1 0.1 1.0734182771900216
Joints:
- joint Torso_BackLowerLeg: origin xyz=0 -2.1939312469491328 0 rpy=0 0 0 -> xyz=0 -1.908138372914677 0 rpy=0 0 0
- joint Torso_FrontLowerLeg: origin xyz=0 1.87378661599641 0 rpy=0 0 0 -> xyz=0 1.908138372914677 0 rpy=0 0 0
- joint Torso_LeftLowerLeg: origin xyz=-1.9329689913046473 0 0 rpy=0 0 0 -> xyz=-1.8002263045399527 0 0 rpy=0 0 0
- joint Torso_RightLowerLeg: origin xyz=2.189386120419314 0 0 rpy=0 0 0 -> xyz=1.8002263045399527 0 0 rpy=0 0 0

File: body16.urdf (robot description, URDF)
Before this commit: robot robot, 9 links, 8 joints
Links:
- link BackLeg: geometry collision box size=0.3166310574724504 2.131583251994387 0.1670597600853507; visual box size=0.3166310574724504 2.131583251994387 0.1670597600853507
- link BackLowerLeg: geometry collision box size=0.2267900209300976 0.1 1.0235398341114677; visual box size=0.2267900209300976 0.1 1.0235398341114677
- link FrontLeg: geometry collision box size=0.3166310574724504 2.131583251994387 0.1670597600853507; visual box size=0.3166310574724504 2.131583251994387 0.1670597600853507
- link FrontLowerLeg: geometry collision box size=0.2267900209300976 0.1 1.0235398341114677; visual box size=0.2267900209300976 0.1 1.0235398341114677
- link LeftLeg: geometry collision box size=1.927182230518755 0.3068481334992934 0.36154173739017476; visual box size=1.927182230518755 0.3068481334992934 0.36154173739017476
- link LeftLowerLeg: geometry collision box size=0.3063950048641242 0.26294403541808625 0.8241496519936401; visual box size=0.3063950048641242 0.26294403541808625 0.8241496519936401
- link RightLeg: geometry collision box size=1.927182230518755 0.3068481334992934 0.36154173739017476; visual box size=1.927182230518755 0.3068481334992934 0.36154173739017476
- link RightLowerLeg: geometry collision box size=0.3063950048641242 0.26294403541808625 0.8241496519936401; visual box size=0.3063950048641242 0.26294403541808625 0.8241496519936401
Joints:
- joint Torso_BackLowerLeg: origin xyz=0 -2.022054594580288 0 rpy=0 0 0 -> xyz=0 -2.131583251994387 0 rpy=0 0 0
- joint Torso_FrontLowerLeg: origin xyz=0 1.9838907702629909 0 rpy=0 0 0 -> xyz=0 2.131583251994387 0 rpy=0 0 0
- joint Torso_LeftLowerLeg: origin xyz=-1.9539942673073993 0 0 rpy=0 0 0 -> xyz=-1.927182230518755 0 0 rpy=0 0 0
- joint Torso_RightLowerLeg: origin xyz=2.1004210868661497 0 0 rpy=0 0 0 -> xyz=1.927182230518755 0 0 rpy=0 0 0

File: body17.urdf (robot description, URDF)
Before this commit: robot robot, 9 links, 8 joints
Links:
- link BackLeg: geometry collision box size=0.3818612482594608 1.8124232551033117 0.14934569812542522; visual box size=0.3818612482594608 1.8124232551033117 0.14934569812542522
- link BackLowerLeg: geometry collision box size=0.1 0.44014955395554367 1.1857322973397615; visual box size=0.1 0.44014955395554367 1.1857322973397615
- link FrontLeg: geometry collision box size=0.3818612482594608 1.8124232551033117 0.14934569812542522; visual box size=0.3818612482594608 1.8124232551033117 0.14934569812542522
- link FrontLowerLeg: geometry collision box size=0.1 0.44014955395554367 1.1857322973397615; visual box size=0.1 0.44014955395554367 1.1857322973397615
- link LeftLeg: geometry collision box size=1.962431265231472 0.20561102607705878 0.14999249035266762; visual box size=1.962431265231472 0.20561102607705878 0.14999249035266762
- link LeftLowerLeg: geometry collision box size=0.2818917813228853 0.2951205848626923 1.0783185945741063; visual box size=0.2818917813228853 0.2951205848626923 1.0783185945741063
- link RightLeg: geometry collision box size=1.962431265231472 0.20561102607705878 0.14999249035266762; visual box size=1.962431265231472 0.20561102607705878 0.14999249035266762
- link RightLowerLeg: geometry collision box size=0.2818917813228853 0.2951205848626923 1.0783185945741063; visual box size=0.2818917813228853 0.2951205848626923 1.0783185945741063
Joints:
- joint Torso_BackLowerLeg: origin xyz=0 -1.8298010697276819 0 rpy=0 0 0 -> xyz=0 -1.8124232551033117 0 rpy=0 0 0
- joint Torso_FrontLowerLeg: origin xyz=0 2.0049392177492793 0 rpy=0 0 0 -> xyz=0 1.8124232551033117 0 rpy=0 0 0
- joint Torso_LeftLowerLeg: origin xyz=-2.0231558906735363 0 0 rpy=0 0 0 -> xyz=-1.962431265231472 0 0 rpy=0 0 0
- joint Torso_RightLowerLeg: origin xyz=2.0810971880567735 0 0 rpy=0 0 0 -> xyz=1.962431265231472 0 0 rpy=0 0 0

File: body18.urdf (robot description, URDF)
Before this commit: robot robot, 9 links, 8 joints
Links:
- link BackLeg: geometry collision box size=0.10807764821708812 1.9521552097028196 0.38204070201060325; visual box size=0.10807764821708812 1.9521552097028196 0.38204070201060325
- link BackLowerLeg: geometry collision box size=0.2304353835827079 0.1 1.0806913169252161; visual box size=0.2304353835827079 0.1 1.0806913169252161
- link FrontLeg: geometry collision box size=0.10807764821708812 1.9521552097028196 0.38204070201060325; visual box size=0.10807764821708812 1.9521552097028196 0.38204070201060325
- link FrontLowerLeg: geometry collision box size=0.2304353835827079 0.1 1.0806913169252161; visual box size=0.2304353835827079 0.1 1.0806913169252161
- link LeftLeg: geometry collision box size=1.9784483417280538 0.3546336911726484 0.29634539849396185; visual box size=1.9784483417280538 0.3546336911726484 0.29634539849396185
- link LeftLowerLeg: geometry collision box size=0.3555063014211877 0.1 1.19773028212462; visual box size=0.3555063014211877 0.1 1.19773028212462
- link RightLeg: geometry collision box size=1.9784483417280538 0.3546336911726484 0.29634539849396185; visual box size=1.9784483417280538 0.3546336911726484 0.29634539849396185
- link RightLowerLeg: geometry collision box size=0.3555063014211877 0.1 1.19773028212462; visual box size=0.3555063014211877 0.1 1.19773028212462
Joints:
- joint Torso_BackLowerLeg: origin xyz=0 -2.0379111331992266 0 rpy=0 0 0 -> xyz=0 -1.9521552097028196 0 rpy=0 0 0
- joint Torso_FrontLowerLeg: origin xyz=0 1.8500609095755756 0 rpy=0 0 0 -> xyz=0 1.9521552097028196 0 rpy=0 0 0
- joint Torso_LeftLowerLeg: origin xyz=-2.076820669576879 0 0 rpy=0 0 0 -> xyz=-1.9784483417280538 0 0 rpy=0 0 0
- joint Torso_RightLowerLeg: origin xyz=1.9198077672482432 0 0 rpy=0 0 0 -> xyz=1.9784483417280538 0 0 rpy=0 0 0

File: body19.urdf (robot description, URDF)
Before this commit: robot robot, 9 links, 8 joints
Links:
- link BackLeg: geometry collision box size=0.17990255908863334 2.221926997162531 0.1381713292150013; visual box size=0.17990255908863334 2.221926997162531 0.1381713292150013
- link BackLowerLeg: geometry collision box size=0.15715363293877052 0.24038749782715477 0.9713038595495024; visual box size=0.15715363293877052 0.24038749782715477 0.9713038595495024
- link FrontLeg: geometry collision box size=0.17990255908863334 2.221926997162531 0.1381713292150013; visual box size=0.17990255908863334 2.221926997162531 0.1381713292150013
- link FrontLowerLeg: geometry collision box size=0.15715363293877052 0.24038749782715477 0.9713038595495024; visual box size=0.15715363293877052 0.24038749782715477 0.9713038595495024
- link LeftLeg: geometry collision box size=1.831290686135426 0.3012412223233153 0.22874491764993468; visual box size=1.831290686135426 0.3012412223233153 0.22874491764993468
- link LeftLowerLeg: geometry collision box size=0.30028169364072377 0.1579222058371365 1.0386421926267424; visual box size=0.30028169364072377 0.1579222058371365 1.0386421926267424
- link RightLeg: geometry collision box size=1.831290686135426 0.3012412223233153 0.22874491764993468; visual box size=1.831290686135426 0.3012412223233153 0.22874491764993468
- link RightLowerLeg: geometry collision box size=0.30028169364072377 0.1579222058371365 1.0386421926267424; visual box size=0.30028169364072377 0.1579222058371365 1.0386421926267424
Joints:
- joint Torso_BackLowerLeg: origin xyz=0 -2.1272600016630983 0 rpy=0 0 0 -> xyz=0 -2.221926997162531 0 rpy=0 0 0
- joint Torso_FrontLowerLeg: origin xyz=0 2.0595484327803613 0 rpy=0 0 0 -> xyz=0 2.221926997162531 0 rpy=0 0 0
- joint Torso_LeftLowerLeg: origin xyz=-1.8617840327082285 0 0 rpy=0 0 0 -> xyz=-1.831290686135426 0 0 rpy=0 0 0
- joint Torso_RightLowerLeg: origin xyz=1.8383179420195954 0 0 rpy=0 0 0 -> xyz=1.831290686135426 0 0 rpy=0 0 0

File: body20.urdf (robot description, URDF)
Before this commit: robot robot, 9 links, 8 joints
Links:
- link BackLeg: geometry collision box size=0.1 2.0948417418807437 0.2538254234506498; visual box size=0.1 2.0948417418807437 0.2538254234506498
- link BackLowerLeg: geometry collision box size=0.24256220359822944 0.1 0.9719102612742614; visual box size=0.24256220359822944 0.1 0.9719102612742614
- link FrontLeg: geometry collision box size=0.1 2.0948417418807437 0.2538254234506498; visual box size=0.1 2.0948417418807437 0.2538254234506498
- link FrontLowerLeg: geometry collision box size=0.24256220359822944 0.1 0.9719102612742614; visual box size=0.24256220359822944 0.1 0.9719102612742614
- link LeftLeg: geometry collision box size=1.845254525118026 0.3707687763520635 0.3353591775186319; visual box size=1.845254525118026 0.3707687763520635 0.3353591775186319
- link LeftLowerLeg: geometry collision box size=0.21927050773505674 0.24698512653823268 1.067963905523416; visual box size=0.21927050773505674 0.24698512653823268 1.067963905523416
- link RightLeg: geometry collision box size=1.845254525118026 0.3707687763520635 0.3353591775186319; visual box size=1.845254525118026 0.3707687763520635 0.3353591775186319
- link RightLowerLeg: geometry collision box size=0.21927050773505674 0.24698512653823268 1.067963905523416; visual box size=0.21927050773505674 0.24698512653823268 1.067963905523416
Joints:
- joint Torso_BackLowerLeg: origin xyz=0 -1.9364981682877995 0 rpy=0 0 0 -> xyz=0 -2.0948417418807437 0 rpy=0 0 0
- joint Torso_FrontLowerLeg: origin xyz=0 2.183242900429535 0 rpy=0 0 0 -> xyz=0 2.0948417418807437 0 rpy=0 0 0
- joint Torso_LeftLowerLeg: origin xyz=-1.8035698297439704 0 0 rpy=0 0 0 -> xyz=-1.845254525118026 0 0 rpy=0 0 0
- joint Torso_RightLowerLeg: origin xyz=1.807508959756891 0 0 rpy=0 0 0 -> xyz=1.845254525118026 0 0 rpy=0 0 0

File: body21.urdf (robot description, URDF)
Before this commit: robot robot, 9 links, 8 joints
Links:
- link BackLeg: geometry collision box size=0.1 1.8795610506714615 0.1; visual box size=0.1 1.8795610506714615 0.1
- link BackLowerLeg: geometry collision box size=0.1 0.1 1.1041517849905724; visual box size=0.1 0.1 1.1041517849905724
- link FrontLeg: geometry collision box size=0.1 1.8795610506714615 0.1; visual box size=0.1 1.8795610506714615 0.1
- link FrontLowerLeg: geometry collision box size=0.1 0.1 1.1041517849905724; visual box size=0.1 0.1 1.1041517849905724
- link LeftLeg: geometry collision box size=1.8055839773827302 0.3239718937363843 0.1; visual box size=1.8055839773827302 0.3239718937363843 0.1
- link LeftLowerLeg: geometry collision box size=0.1300189675472665 0.29618196855389073 0.9158182927327438; visual box size=0.1300189675472665 0.29618196855389073 0.9158182927327438
- link RightLeg: geometry collision box size=1.8055839773827302 0.3239718937363843 0.1; visual box size=1.8055839773827302 0.3239718937363843 0.1
- link RightLowerLeg: geometry collision box size=0.1300189675472665 0.29618196855389073 0.9158182927327438; visual box size=0.1300189675472665 0.29618196855389073 0.9158182927327438
Joints:
- joint Torso_BackLowerLeg: origin xyz=0 -2.1470884840853905 0 rpy=0 0 0 -> xyz=0 -1.8795610506714615 0 rpy=0 0 0
- joint Torso_FrontLowerLeg: origin xyz=0 2.0006453836484 0 rpy=0 0 0 -> xyz=0 1.8795610506714615 0 rpy=0 0 0
- joint Torso_LeftLowerLeg: origin xyz=-1.8463876560165389 0 0 rpy=0 0 0 -> xyz=-1.8055839773827302 0 0 rpy=0 0 0
- joint Torso_RightLowerLeg: origin xyz=2.0117398345936945 0 0 rpy=0 0 0 -> xyz=1.8055839773827302 0 0 rpy=0 0 0
