Commit message: symmetry added

File: body22.urdf (robot description, URDF)
Before this commit: robot robot, 9 links, 8 joints
Links:
- link BackLeg: geometry collision box size=0.22340406220199102 1.9006395926468471 0.1; visual box size=0.22340406220199102 1.9006395926468471 0.1
- link BackLowerLeg: geometry collision box size=0.1 0.43170217210707645 1.281792291339208; visual box size=0.1 0.43170217210707645 1.281792291339208
- link FrontLeg: geometry collision box size=0.22340406220199102 1.9006395926468471 0.1; visual box size=0.22340406220199102 1.9006395926468471 0.1
- link FrontLowerLeg: geometry collision box size=0.1 0.43170217210707645 1.281792291339208; visual box size=0.1 0.43170217210707645 1.281792291339208
- link LeftLeg: geometry collision box size=1.9311245312409582 0.1 0.40405057001658623; visual box size=1.9311245312409582 0.1 0.40405057001658623
- link LeftLowerLeg: geometry collision box size=0.24048907153705842 0.48617405801780905 1.1615282412490797; visual box size=0.24048907153705842 0.48617405801780905 1.1615282412490797
- link RightLeg: geometry collision box size=1.9311245312409582 0.1 0.40405057001658623; visual box size=1.9311245312409582 0.1 0.40405057001658623
- link RightLowerLeg: geometry collision box size=0.24048907153705842 0.48617405801780905 1.1615282412490797; visual box size=0.24048907153705842 0.48617405801780905 1.1615282412490797
Joints:
- joint Torso_BackLowerLeg: origin xyz=0 -1.9519985311512655 0 rpy=0 0 0 -> xyz=0 -1.9006395926468471 0 rpy=0 0 0
- joint Torso_FrontLowerLeg: origin xyz=0 2.017346313765154 0 rpy=0 0 0 -> xyz=0 1.9006395926468471 0 rpy=0 0 0
- joint Torso_LeftLowerLeg: origin xyz=-1.9592047876863252 0 0 rpy=0 0 0 -> xyz=-1.9311245312409582 0 0 rpy=0 0 0
- joint Torso_RightLowerLeg: origin xyz=2.1708933615222663 0 0 rpy=0 0 0 -> xyz=1.9311245312409582 0 0 rpy=0 0 0

File: body23.urdf (robot description, URDF)
Before this commit: robot robot, 9 links, 8 joints
Links:
- link BackLeg: geometry collision box size=0.1 2.177081201168779 0.1; visual box size=0.1 2.177081201168779 0.1
- link BackLowerLeg: geometry collision box size=0.22075312146010817 0.34702477725160774 1.1617538902863407; visual box size=0.22075312146010817 0.34702477725160774 1.1617538902863407
- link FrontLeg: geometry collision box size=0.1 2.177081201168779 0.1; visual box size=0.1 2.177081201168779 0.1
- link FrontLowerLeg: geometry collision box size=0.22075312146010817 0.34702477725160774 1.1617538902863407; visual box size=0.22075312146010817 0.34702477725160774 1.1617538902863407
- link LeftLeg: geometry collision box size=2.0083836864552107 0.18642126335268072 0.12920295107714327; visual box size=2.0083836864552107 0.18642126335268072 0.12920295107714327
- link LeftLowerLeg: geometry collision box size=0.3069173489573921 0.1782706887780622 1.1598249267513179; visual box size=0.3069173489573921 0.1782706887780622 1.1598249267513179
- link RightLeg: geometry collision box size=2.0083836864552107 0.18642126335268072 0.12920295107714327; visual box size=2.0083836864552107 0.18642126335268072 0.12920295107714327
- link RightLowerLeg: geometry collision box size=0.3069173489573921 0.1782706887780622 1.1598249267513179; visual box size=0.3069173489573921 0.1782706887780622 1.1598249267513179
Joints:
- joint Torso_BackLowerLeg: origin xyz=0 -2.110659374906141 0 rpy=0 0 0 -> xyz=0 -2.177081201168779 0 rpy=0 0 0
- joint Torso_FrontLowerLeg: origin xyz=0 1.833995850994513 0 rpy=0 0 0 -> xyz=0 2.177081201168779 0 rpy=0 0 0
- joint Torso_LeftLowerLeg: origin xyz=-2.125487039516252 0 0 rpy=0 0 0 -> xyz=-2.0083836864552107 0 0 rpy=0 0 0
- joint Torso_RightLowerLeg: origin xyz=1.963131823315977 0 0 rpy=0 0 0 -> xyz=2.0083836864552107 0 0 rpy=0 0 0

File: body24.urdf (robot description, URDF)
Before this commit: robot robot, 9 links, 8 joints
Links:
- link BackLeg: geometry collision box size=0.2821695632288598 2.19972151574263 0.1; visual box size=0.2821695632288598 2.19972151574263 0.1
- link BackLowerLeg: geometry collision box size=0.2025053815841966 0.3858124011664692 0.9100003420155659; visual box size=0.2025053815841966 0.3858124011664692 0.9100003420155659
- link FrontLeg: geometry collision box size=0.2821695632288598 2.19972151574263 0.1; visual box size=0.2821695632288598 2.19972151574263 0.1
- link FrontLowerLeg: geometry collision box size=0.2025053815841966 0.3858124011664692 0.9100003420155659; visual box size=0.2025053815841966 0.3858124011664692 0.9100003420155659
- link LeftLeg: geometry collision box size=2.024105548797988 0.15853668598796872 0.1510648453426703; visual box size=2.024105548797988 0.15853668598796872 0.1510648453426703
- link LeftLowerLeg: geometry collision box size=0.16114652840214816 0.1 0.9192736307250945; visual box size=0.16114652840214816 0.1 0.9192736307250945
- link RightLeg: geometry collision box size=2.024105548797988 0.15853668598796872 0.1510648453426703; visual box size=2.024105548797988 0.15853668598796872 0.1510648453426703
- link RightLowerLeg: geometry collision box size=0.16114652840214816 0.1 0.9192736307250945; visual box size=0.16114652840214816 0.1 0.9192736307250945
Joints:
- joint Torso_BackLowerLeg: origin xyz=0 -1.986106833459668 0 rpy=0 0 0 -> xyz=0 -2.19972151574263 0 rpy=0 0 0
- joint Torso_FrontLowerLeg: origin xyz=0 2.02482773202148 0 rpy=0 0 0 -> xyz=0 2.19972151574263 0 rpy=0 0 0
- joint Torso_LeftLowerLeg: origin xyz=-1.8644932884187058 0 0 rpy=0 0 0 -> xyz=-2.024105548797988 0 0 rpy=0 0 0
- joint Torso_RightLowerLeg: origin xyz=2.0227876957225055 0 0 rpy=0 0 0 -> xyz=2.024105548797988 0 0 rpy=0 0 0

File: body25.urdf (robot description, URDF)
Before this commit: robot robot, 9 links, 8 joints
Links:
- link BackLeg: geometry collision box size=0.1 1.9769062200278906 0.15374468291679405; visual box size=0.1 1.9769062200278906 0.15374468291679405
- link BackLowerLeg: geometry collision box size=0.34702370204531247 0.23763912294970843 1.0360007940323306; visual box size=0.34702370204531247 0.23763912294970843 1.0360007940323306
- link FrontLeg: geometry collision box size=0.1 1.9769062200278906 0.15374468291679405; visual box size=0.1 1.9769062200278906 0.15374468291679405
- link FrontLowerLeg: geometry collision box size=0.34702370204531247 0.23763912294970843 1.0360007940323306; visual box size=0.34702370204531247 0.23763912294970843 1.0360007940323306
- link LeftLeg: geometry collision box size=1.952052715475317 0.22852541818489608 0.2990622081334315; visual box size=1.952052715475317 0.22852541818489608 0.2990622081334315
- link LeftLowerLeg: geometry collision box size=0.28781156450116296 0.15130238370796617 1.155417727555935; visual box size=0.28781156450116296 0.15130238370796617 1.155417727555935
- link RightLeg: geometry collision box size=1.952052715475317 0.22852541818489608 0.2990622081334315; visual box size=1.952052715475317 0.22852541818489608 0.2990622081334315
- link RightLowerLeg: geometry collision box size=0.28781156450116296 0.15130238370796617 1.155417727555935; visual box size=0.28781156450116296 0.15130238370796617 1.155417727555935
Joints:
- joint Torso_BackLowerLeg: origin xyz=0 -2.0457676745248485 0 rpy=0 0 0 -> xyz=0 -1.9769062200278906 0 rpy=0 0 0
- joint Torso_FrontLowerLeg: origin xyz=0 2.1127764126012427 0 rpy=0 0 0 -> xyz=0 1.9769062200278906 0 rpy=0 0 0
- joint Torso_LeftLowerLeg: origin xyz=-2.004481711407217 0 0 rpy=0 0 0 -> xyz=-1.952052715475317 0 0 rpy=0 0 0
- joint Torso_RightLowerLeg: origin xyz=1.8785878784868746 0 0 rpy=0 0 0 -> xyz=1.952052715475317 0 0 rpy=0 0 0

File: body26.urdf (robot description, URDF)
Before this commit: robot robot, 9 links, 8 joints
Links:
- link BackLeg: geometry collision box size=0.13667778333091044 2.083439347529 0.1; visual box size=0.13667778333091044 2.083439347529 0.1
- link BackLowerLeg: geometry collision box size=0.30564019114415053 0.2205839304728753 0.8694333674156348; visual box size=0.30564019114415053 0.2205839304728753 0.8694333674156348
- link FrontLeg: geometry collision box size=0.13667778333091044 2.083439347529 0.1; visual box size=0.13667778333091044 2.083439347529 0.1
- link FrontLowerLeg: geometry collision box size=0.30564019114415053 0.2205839304728753 0.8694333674156348; visual box size=0.30564019114415053 0.2205839304728753 0.8694333674156348
- link LeftLeg: geometry collision box size=1.814803256340219 0.1 0.1; visual box size=1.814803256340219 0.1 0.1
- link LeftLowerLeg: geometry collision box size=0.18914325683326721 0.3127630117094558 1.096341099243014; visual box size=0.18914325683326721 0.3127630117094558 1.096341099243014
- link RightLeg: geometry collision box size=1.814803256340219 0.1 0.1; visual box size=1.814803256340219 0.1 0.1
- link RightLowerLeg: geometry collision box size=0.18914325683326721 0.3127630117094558 1.096341099243014; visual box size=0.18914325683326721 0.3127630117094558 1.096341099243014
Joints:
- joint Torso_BackLowerLeg: origin xyz=0 -1.8438680260929938 0 rpy=0 0 0 -> xyz=0 -2.083439347529 0 rpy=0 0 0
- joint Torso_FrontLowerLeg: origin xyz=0 1.899533957341911 0 rpy=0 0 0 -> xyz=0 2.083439347529 0 rpy=0 0 0
- joint Torso_LeftLowerLeg: origin xyz=-2.0348399745970034 0 0 rpy=0 0 0 -> xyz=-1.814803256340219 0 0 rpy=0 0 0
- joint Torso_RightLowerLeg: origin xyz=2.1201127648670175 0 0 rpy=0 0 0 -> xyz=1.814803256340219 0 0 rpy=0 0 0

File: body27.urdf (robot description, URDF)
Before this commit: robot robot, 9 links, 8 joints
Links:
- link BackLeg: geometry collision box size=0.18860605835000846 1.8470312269087545 0.1947381810953249; visual box size=0.18860605835000846 1.8470312269087545 0.1947381810953249
- link BackLowerLeg: geometry collision box size=0.1 0.5733533874972794 1.182617493420732; visual box size=0.1 0.5733533874972794 1.182617493420732
- link FrontLeg: geometry collision box size=0.18860605835000846 1.8470312269087545 0.1947381810953249; visual box size=0.18860605835000846 1.8470312269087545 0.1947381810953249
- link FrontLowerLeg: geometry collision box size=0.1 0.5733533874972794 1.182617493420732; visual box size=0.1 0.5733533874972794 1.182617493420732
- link LeftLeg: geometry collision box size=1.917229370844435 0.1 0.5116743143893265; visual box size=1.917229370844435 0.1 0.5116743143893265
- link LeftLowerLeg: geometry collision box size=0.1 0.5732241595130725 1.0790926134476608; visual box size=0.1 0.5732241595130725 1.0790926134476608
- link RightLeg: geometry collision box size=1.917229370844435 0.1 0.5116743143893265; visual box size=1.917229370844435 0.1 0.5116743143893265
- link RightLowerLeg: geometry collision box size=0.1 0.5732241595130725 1.0790926134476608; visual box size=0.1 0.5732241595130725 1.0790926134476608
Joints:
- joint Torso_BackLowerLeg: origin xyz=0 -2.1880817049671153 0 rpy=0 0 0 -> xyz=0 -1.8470312269087545 0 rpy=0 0 0
- joint Torso_FrontLowerLeg: origin xyz=0 1.8405439882645762 0 rpy=0 0 0 -> xyz=0 1.8470312269087545 0 rpy=0 0 0
- joint Torso_LeftLowerLeg: origin xyz=-2.11103705271834 0 0 rpy=0 0 0 -> xyz=-1.917229370844435 0 0 rpy=0 0 0
- joint Torso_RightLowerLeg: origin xyz=2.107388304375555 0 0 rpy=0 0 0 -> xyz=1.917229370844435 0 0 rpy=0 0 0

File: body28.urdf (robot description, URDF)
Before this commit: robot robot, 9 links, 8 joints
Links:
- link BackLeg: geometry collision box size=0.1 2.091513519679978 0.2931677175745251; visual box size=0.1 2.091513519679978 0.2931677175745251
- link BackLowerLeg: geometry collision box size=0.1918398531686633 0.260992561819891 1.2232276708761909; visual box size=0.1918398531686633 0.260992561819891 1.2232276708761909
- link FrontLeg: geometry collision box size=0.1 2.091513519679978 0.2931677175745251; visual box size=0.1 2.091513519679978 0.2931677175745251
- link FrontLowerLeg: geometry collision box size=0.1918398531686633 0.260992561819891 1.2232276708761909; visual box size=0.1918398531686633 0.260992561819891 1.2232276708761909
- link LeftLeg: geometry collision box size=1.8397547740281959 0.1972296621355883 0.14827621341591601; visual box size=1.8397547740281959 0.1972296621355883 0.14827621341591601
- link LeftLowerLeg: geometry collision box size=0.450799226775669 0.1 1.0602786271608167; visual box size=0.450799226775669 0.1 1.0602786271608167
- link RightLeg: geometry collision box size=1.8397547740281959 0.1972296621355883 0.14827621341591601; visual box size=1.8397547740281959 0.1972296621355883 0.14827621341591601
- link RightLowerLeg: geometry collision box size=0.450799226775669 0.1 1.0602786271608167; visual box size=0.450799226775669 0.1 1.0602786271608167
Joints:
- joint Torso_BackLowerLeg: origin xyz=0 -1.995100287677448 0 rpy=0 0 0 -> xyz=0 -2.091513519679978 0 rpy=0 0 0
- joint Torso_FrontLowerLeg: origin xyz=0 2.1645712640676695 0 rpy=0 0 0 -> xyz=0 2.091513519679978 0 rpy=0 0 0
- joint Torso_LeftLowerLeg: origin xyz=-2.04055255798058 0 0 rpy=0 0 0 -> xyz=-1.8397547740281959 0 0 rpy=0 0 0
- joint Torso_RightLowerLeg: origin xyz=2.1446244684085873 0 0 rpy=0 0 0 -> xyz=1.8397547740281959 0 0 rpy=0 0 0

File: body29.urdf (robot description, URDF)
Before this commit: robot robot, 9 links, 8 joints
Links:
- link BackLeg: geometry collision box size=0.23035567129175286 2.0872385847077206 0.1; visual box size=0.23035567129175286 2.0872385847077206 0.1
- link BackLowerLeg: geometry collision box size=0.11976890368400142 0.33754273582419625 0.8786765039935307; visual box size=0.11976890368400142 0.33754273582419625 0.8786765039935307
- link FrontLeg: geometry collision box size=0.23035567129175286 2.0872385847077206 0.1; visual box size=0.23035567129175286 2.0872385847077206 0.1
- link FrontLowerLeg: geometry collision box size=0.11976890368400142 0.33754273582419625 0.8786765039935307; visual box size=0.11976890368400142 0.33754273582419625 0.8786765039935307
- link LeftLeg: geometry collision box size=1.9450566545074963 0.1 0.11204109395519457; visual box size=1.9450566545074963 0.1 0.11204109395519457
- link LeftLowerLeg: geometry collision box size=0.1 0.1 0.9375362568118811; visual box size=0.1 0.1 0.9375362568118811
- link RightLeg: geometry collision box size=1.9450566545074963 0.1 0.11204109395519457; visual box size=1.9450566545074963 0.1 0.11204109395519457
- link RightLowerLeg: geometry collision box size=0.1 0.1 0.9375362568118811; visual box size=0.1 0.1 0.9375362568118811
Joints:
- joint Torso_BackLowerLeg: origin xyz=0 -2.064927769614691 0 rpy=0 0 0 -> xyz=0 -2.0872385847077206 0 rpy=0 0 0
- joint Torso_FrontLowerLeg: origin xyz=0 2.1696218344534137 0 rpy=0 0 0 -> xyz=0 2.0872385847077206 0 rpy=0 0 0
- joint Torso_LeftLowerLeg: origin xyz=-1.8090888427351475 0 0 rpy=0 0 0 -> xyz=-1.9450566545074963 0 0 rpy=0 0 0
- joint Torso_RightLowerLeg: origin xyz=2.0327803462204486 0 0 rpy=0 0 0 -> xyz=1.9450566545074963 0 0 rpy=0 0 0
