Commit message: milestone 4 done

File: body10.urdf (robot description, URDF)
Before this commit: robot robot, 9 links, 8 joints
Links:
- link BackLeg: geometry collision box size=0.2 2 0.2; visual box size=0.2 2 0.2
- link BackLowerLeg: geometry collision box size=0.2 0.2 1; visual box size=0.2 0.2 1
- link FrontLeg: geometry collision box size=0.2 2 0.2; visual box size=0.2 2 0.2
- link FrontLowerLeg: geometry collision box size=0.2 0.2 1; visual box size=0.2 0.2 1
- link LeftLeg: geometry collision box size=2 0.2 0.2; visual box size=2 0.2 0.2
- link LeftLowerLeg: geometry collision box size=0.2 0.2 1; visual box size=0.2 0.2 1
- link RightLeg: geometry collision box size=2 0.2 0.2; visual box size=2 0.2 0.2
- link RightLowerLeg: geometry collision box size=0.2 0.2 1; visual box size=0.2 0.2 1
Joints:
- joint Torso_BackLowerLeg: origin xyz=0 -1.8767691195714171 0 rpy=0 0 0 -> xyz=0 -2 0 rpy=0 0 0
- joint Torso_FrontLowerLeg: origin xyz=0 1.8767691195714171 0 rpy=0 0 0 -> xyz=0 2 0 rpy=0 0 0
- joint Torso_LeftLowerLeg: origin xyz=-2.110298966186739 0 0 rpy=0 0 0 -> xyz=-2 0 0 rpy=0 0 0
- joint Torso_RightLowerLeg: origin xyz=2.110298966186739 0 0 rpy=0 0 0 -> xyz=2 0 0 rpy=0 0 0

File: body11.urdf (robot description, URDF)
Before this commit: robot robot, 9 links, 8 joints
Links:
- link BackLeg: geometry collision box size=0.2 2 0.2; visual box size=0.2 2 0.2
- link BackLowerLeg: geometry collision box size=0.2 0.2 1; visual box size=0.2 0.2 1
- link FrontLeg: geometry collision box size=0.2 2 0.2; visual box size=0.2 2 0.2
- link FrontLowerLeg: geometry collision box size=0.2 0.2 1; visual box size=0.2 0.2 1
- link LeftLeg: geometry collision box size=2 0.2 0.2; visual box size=2 0.2 0.2
- link LeftLowerLeg: geometry collision box size=0.2 0.2 1; visual box size=0.2 0.2 1
- link RightLeg: geometry collision box size=2 0.2 0.2; visual box size=2 0.2 0.2
- link RightLowerLeg: geometry collision box size=0.2 0.2 1; visual box size=0.2 0.2 1
Joints:
- joint Torso_BackLowerLeg: origin xyz=0 -1.9017698948772108 0 rpy=0 0 0 -> xyz=0 -2 0 rpy=0 0 0
- joint Torso_FrontLowerLeg: origin xyz=0 1.9017698948772108 0 rpy=0 0 0 -> xyz=0 2 0 rpy=0 0 0
- joint Torso_LeftLowerLeg: origin xyz=-2.111003577918722 0 0 rpy=0 0 0 -> xyz=-2 0 0 rpy=0 0 0
- joint Torso_RightLowerLeg: origin xyz=2.111003577918722 0 0 rpy=0 0 0 -> xyz=2 0 0 rpy=0 0 0

File: body12.urdf (robot description, URDF)
Before this commit: robot robot, 9 links, 8 joints
Links:
- link BackLeg: geometry collision box size=0.2 2 0.2; visual box size=0.2 2 0.2
- link BackLowerLeg: geometry collision box size=0.2 0.2 1; visual box size=0.2 0.2 1
- link FrontLeg: geometry collision box size=0.2 2 0.2; visual box size=0.2 2 0.2
- link FrontLowerLeg: geometry collision box size=0.2 0.2 1; visual box size=0.2 0.2 1
- link LeftLeg: geometry collision box size=2 0.2 0.2; visual box size=2 0.2 0.2
- link LeftLowerLeg: geometry collision box size=0.2 0.2 1; visual box size=0.2 0.2 1
- link RightLeg: geometry collision box size=2 0.2 0.2; visual box size=2 0.2 0.2
- link RightLowerLeg: geometry collision box size=0.2 0.2 1; visual box size=0.2 0.2 1
Joints:
- joint Torso_BackLowerLeg: origin xyz=0 -1.8623866089559789 0 rpy=0 0 0 -> xyz=0 -2 0 rpy=0 0 0
- joint Torso_FrontLowerLeg: origin xyz=0 1.8623866089559789 0 rpy=0 0 0 -> xyz=0 2 0 rpy=0 0 0
- joint Torso_LeftLowerLeg: origin xyz=-1.878309033324971 0 0 rpy=0 0 0 -> xyz=-2 0 0 rpy=0 0 0
- joint Torso_RightLowerLeg: origin xyz=1.878309033324971 0 0 rpy=0 0 0 -> xyz=2 0 0 rpy=0 0 0

File: body13.urdf (robot description, URDF)
Before this commit: robot robot, 9 links, 8 joints
Links:
- link BackLeg: geometry collision box size=0.2 2 0.2; visual box size=0.2 2 0.2
- link BackLowerLeg: geometry collision box size=0.2 0.2 1; visual box size=0.2 0.2 1
- link FrontLeg: geometry collision box size=0.2 2 0.2; visual box size=0.2 2 0.2
- link FrontLowerLeg: geometry collision box size=0.2 0.2 1; visual box size=0.2 0.2 1
- link LeftLeg: geometry collision box size=2 0.2 0.2; visual box size=2 0.2 0.2
- link LeftLowerLeg: geometry collision box size=0.2 0.2 1; visual box size=0.2 0.2 1
- link RightLeg: geometry collision box size=2 0.2 0.2; visual box size=2 0.2 0.2
- link RightLowerLeg: geometry collision box size=0.2 0.2 1; visual box size=0.2 0.2 1
Joints:
- joint Torso_BackLowerLeg: origin xyz=0 -2.026237450058545 0 rpy=0 0 0 -> xyz=0 -2 0 rpy=0 0 0
- joint Torso_FrontLowerLeg: origin xyz=0 2.026237450058545 0 rpy=0 0 0 -> xyz=0 2 0 rpy=0 0 0
- joint Torso_LeftLowerLeg: origin xyz=-2.0864836820466373 0 0 rpy=0 0 0 -> xyz=-2 0 0 rpy=0 0 0
- joint Torso_RightLowerLeg: origin xyz=2.0864836820466373 0 0 rpy=0 0 0 -> xyz=2 0 0 rpy=0 0 0

File: body14.urdf (robot description, URDF)
Before this commit: robot robot, 9 links, 8 joints
Links:
- link BackLeg: geometry collision box size=0.2 2 0.2; visual box size=0.2 2 0.2
- link BackLowerLeg: geometry collision box size=0.2 0.2 1; visual box size=0.2 0.2 1
- link FrontLeg: geometry collision box size=0.2 2 0.2; visual box size=0.2 2 0.2
- link FrontLowerLeg: geometry collision box size=0.2 0.2 1; visual box size=0.2 0.2 1
- link LeftLeg: geometry collision box size=2 0.2 0.2; visual box size=2 0.2 0.2
- link LeftLowerLeg: geometry collision box size=0.2 0.2 1; visual box size=0.2 0.2 1
- link RightLeg: geometry collision box size=2 0.2 0.2; visual box size=2 0.2 0.2
- link RightLowerLeg: geometry collision box size=0.2 0.2 1; visual box size=0.2 0.2 1
Joints:
- joint Torso_BackLowerLeg: origin xyz=0 -2.3112030941718085 0 rpy=0 0 0 -> xyz=0 -2 0 rpy=0 0 0
- joint Torso_FrontLowerLeg: origin xyz=0 2.3112030941718085 0 rpy=0 0 0 -> xyz=0 2 0 rpy=0 0 0
- joint Torso_LeftLowerLeg: origin xyz=-1.8940597804259327 0 0 rpy=0 0 0 -> xyz=-2 0 0 rpy=0 0 0
- joint Torso_RightLowerLeg: origin xyz=1.8940597804259327 0 0 rpy=0 0 0 -> xyz=2 0 0 rpy=0 0 0

File: body15.urdf (robot description, URDF)
Before this commit: robot robot, 9 links, 8 joints
Links:
- link BackLeg: geometry collision box size=0.1 2.0038324744462064 0.13321166434828058; visual box size=0.1 2.0038324744462064 0.13321166434828058
- link BackLowerLeg: geometry collision box size=0.24922518394919715 0.24098984252862504 0.8078792574057867; visual box size=0.24922518394919715 0.24098984252862504 0.8078792574057867
- link FrontLeg: geometry collision box size=0.1 2.0038324744462064 0.13321166434828058; visual box size=0.1 2.0038324744462064 0.13321166434828058
- link FrontLowerLeg: geometry collision box size=0.24922518394919715 0.24098984252862504 0.8078792574057867; visual box size=0.24922518394919715 0.24098984252862504 0.8078792574057867
- link LeftLeg: geometry collision box size=2.1640890076795687 0.11355555759275143 0.12398292439267272; visual box size=2.1640890076795687 0.11355555759275143 0.12398292439267272
- link LeftLowerLeg: geometry collision box size=0.18588160043104654 0.33036074019993267 0.9503957430311428; visual box size=0.18588160043104654 0.33036074019993267 0.9503957430311428
- link RightLeg: geometry collision box size=2.1640890076795687 0.11355555759275143 0.12398292439267272; visual box size=2.1640890076795687 0.11355555759275143 0.12398292439267272
- link RightLowerLeg: geometry collision box size=0.18588160043104654 0.33036074019993267 0.9503957430311428; visual box size=0.18588160043104654 0.33036074019993267 0.9503957430311428
Joints:
- joint Torso_BackLowerLeg: origin xyz=0 -1.908138372914677 0 rpy=0 0 0 -> xyz=0 -2.0038324744462064 0 rpy=0 0 0
- joint Torso_FrontLowerLeg: origin xyz=0 1.908138372914677 0 rpy=0 0 0 -> xyz=0 2.0038324744462064 0 rpy=0 0 0
- joint Torso_LeftLowerLeg: origin xyz=-1.8002263045399527 0 0 rpy=0 0 0 -> xyz=-2.1640890076795687 0 0 rpy=0 0 0
- joint Torso_RightLowerLeg: origin xyz=1.8002263045399527 0 0 rpy=0 0 0 -> xyz=2.1640890076795687 0 0 rpy=0 0 0

File: body16.urdf (robot description, URDF)
Before this commit: robot robot, 9 links, 8 joints
Links:
- link BackLeg: geometry collision box size=0.3436189779790245 2.027548772102332 0.35532344878932576; visual box size=0.3436189779790245 2.027548772102332 0.35532344878932576
- link BackLowerLeg: geometry collision box size=0.3043254427259654 0.16994941463754656 1.0753942671232353; visual box size=0.3043254427259654 0.16994941463754656 1.0753942671232353
- link FrontLeg: geometry collision box size=0.3436189779790245 2.027548772102332 0.35532344878932576; visual box size=0.3436189779790245 2.027548772102332 0.35532344878932576
- link FrontLowerLeg: geometry collision box size=0.3043254427259654 0.16994941463754656 1.0753942671232353; visual box size=0.3043254427259654 0.16994941463754656 1.0753942671232353
- link LeftLeg: geometry collision box size=1.9687558498034268 0.173116886061188 0.3517320918480277; visual box size=1.9687558498034268 0.173116886061188 0.3517320918480277
- link LeftLowerLeg: geometry collision box size=0.11735697806034336 0.17050295894532322 0.8700642098393617; visual box size=0.11735697806034336 0.17050295894532322 0.8700642098393617
- link RightLeg: geometry collision box size=1.9687558498034268 0.173116886061188 0.3517320918480277; visual box size=1.9687558498034268 0.173116886061188 0.3517320918480277
- link RightLowerLeg: geometry collision box size=0.11735697806034336 0.17050295894532322 0.8700642098393617; visual box size=0.11735697806034336 0.17050295894532322 0.8700642098393617
Joints:
- joint Torso_BackLowerLeg: origin xyz=0 -2.131583251994387 0 rpy=0 0 0 -> xyz=0 -2.027548772102332 0 rpy=0 0 0
- joint Torso_FrontLowerLeg: origin xyz=0 2.131583251994387 0 rpy=0 0 0 -> xyz=0 2.027548772102332 0 rpy=0 0 0
- joint Torso_LeftLowerLeg: origin xyz=-1.927182230518755 0 0 rpy=0 0 0 -> xyz=-1.9687558498034268 0 0 rpy=0 0 0
- joint Torso_RightLowerLeg: origin xyz=1.927182230518755 0 0 rpy=0 0 0 -> xyz=1.9687558498034268 0 0 rpy=0 0 0

File: body17.urdf (robot description, URDF)
Before this commit: robot robot, 9 links, 8 joints
Links:
- link BackLeg: geometry collision box size=0.12216621786762163 2.0441740684421843 0.1; visual box size=0.12216621786762163 2.0441740684421843 0.1
- link BackLowerLeg: geometry collision box size=0.1 0.13113826928556768 0.8857820703692105; visual box size=0.1 0.13113826928556768 0.8857820703692105
- link FrontLeg: geometry collision box size=0.12216621786762163 2.0441740684421843 0.1; visual box size=0.12216621786762163 2.0441740684421843 0.1
- link FrontLowerLeg: geometry collision box size=0.1 0.13113826928556768 0.8857820703692105; visual box size=0.1 0.13113826928556768 0.8857820703692105
- link LeftLeg: geometry collision box size=2.072184416904061 0.3933956241638776 0.1; visual box size=2.072184416904061 0.3933956241638776 0.1
- link LeftLowerLeg: geometry collision box size=0.36759010627085104 0.22232146587843085 0.9658436529543294; visual box size=0.36759010627085104 0.22232146587843085 0.9658436529543294
- link RightLeg: geometry collision box size=2.072184416904061 0.3933956241638776 0.1; visual box size=2.072184416904061 0.3933956241638776 0.1
- link RightLowerLeg: geometry collision box size=0.36759010627085104 0.22232146587843085 0.9658436529543294; visual box size=0.36759010627085104 0.22232146587843085 0.9658436529543294
Joints:
- joint Torso_BackLowerLeg: origin xyz=0 -1.8124232551033117 0 rpy=0 0 0 -> xyz=0 -2.0441740684421843 0 rpy=0 0 0
- joint Torso_FrontLowerLeg: origin xyz=0 1.8124232551033117 0 rpy=0 0 0 -> xyz=0 2.0441740684421843 0 rpy=0 0 0
- joint Torso_LeftLowerLeg: origin xyz=-1.962431265231472 0 0 rpy=0 0 0 -> xyz=-2.072184416904061 0 0 rpy=0 0 0
- joint Torso_RightLowerLeg: origin xyz=1.962431265231472 0 0 rpy=0 0 0 -> xyz=2.072184416904061 0 0 rpy=0 0 0

File: body18.urdf (robot description, URDF)
Before this commit: robot robot, 9 links, 8 joints
Links:
- link BackLeg: geometry collision box size=0.1537976319979511 1.94569395433575 0.1622144277727121; visual box size=0.1537976319979511 1.94569395433575 0.1622144277727121
- link BackLowerLeg: geometry collision box size=0.3107980661130869 0.231819961011553 1.1357657137745065; visual box size=0.3107980661130869 0.231819961011553 1.1357657137745065
- link FrontLeg: geometry collision box size=0.1537976319979511 1.94569395433575 0.1622144277727121; visual box size=0.1537976319979511 1.94569395433575 0.1622144277727121
- link FrontLowerLeg: geometry collision box size=0.3107980661130869 0.231819961011553 1.1357657137745065; visual box size=0.3107980661130869 0.231819961011553 1.1357657137745065
- link LeftLeg: geometry collision box size=1.836878862596924 0.1 0.11872206697363655; visual box size=1.836878862596924 0.1 0.11872206697363655
- link LeftLowerLeg: geometry collision box size=0.3248828566698502 0.35493660740957256 0.8886736863991284; visual box size=0.3248828566698502 0.35493660740957256 0.8886736863991284
- link RightLeg: geometry collision box size=1.836878862596924 0.1 0.11872206697363655; visual box size=1.836878862596924 0.1 0.11872206697363655
- link RightLowerLeg: geometry collision box size=0.3248828566698502 0.35493660740957256 0.8886736863991284; visual box size=0.3248828566698502 0.35493660740957256 0.8886736863991284
Joints:
- joint Torso_BackLowerLeg: origin xyz=0 -1.9521552097028196 0 rpy=0 0 0 -> xyz=0 -1.94569395433575 0 rpy=0 0 0
- joint Torso_FrontLowerLeg: origin xyz=0 1.9521552097028196 0 rpy=0 0 0 -> xyz=0 1.94569395433575 0 rpy=0 0 0
- joint Torso_LeftLowerLeg: origin xyz=-1.9784483417280538 0 0 rpy=0 0 0 -> xyz=-1.836878862596924 0 0 rpy=0 0 0
- joint Torso_RightLowerLeg: origin xyz=1.9784483417280538 0 0 rpy=0 0 0 -> xyz=1.836878862596924 0 0 rpy=0 0 0

File: body19.urdf (robot description, URDF)
Before this commit: robot robot, 9 links, 8 joints
Links:
- link BackLeg: geometry collision box size=0.13796678996476405 2.0242932765670663 0.3924328844900477; visual box size=0.13796678996476405 2.0242932765670663 0.3924328844900477
- link BackLowerLeg: geometry collision box size=0.311999756533474 0.1274557048112135 1.150420616629238; visual box size=0.311999756533474 0.1274557048112135 1.150420616629238
- link FrontLeg: geometry collision box size=0.13796678996476405 2.0242932765670663 0.3924328844900477; visual box size=0.13796678996476405 2.0242932765670663 0.3924328844900477
- link FrontLowerLeg: geometry collision box size=0.311999756533474 0.1274557048112135 1.150420616629238; visual box size=0.311999756533474 0.1274557048112135 1.150420616629238
- link LeftLeg: geometry collision box size=2.1516290903712636 0.10156847301921933 0.18172172266513598; visual box size=2.1516290903712636 0.10156847301921933 0.18172172266513598
- link LeftLowerLeg: geometry collision box size=0.1 0.3000794648212588 0.9092447255385127; visual box size=0.1 0.3000794648212588 0.9092447255385127
- link RightLeg: geometry collision box size=2.1516290903712636 0.10156847301921933 0.18172172266513598; visual box size=2.1516290903712636 0.10156847301921933 0.18172172266513598
- link RightLowerLeg: geometry collision box size=0.1 0.3000794648212588 0.9092447255385127; visual box size=0.1 0.3000794648212588 0.9092447255385127
Joints:
- joint Torso_BackLowerLeg: origin xyz=0 -2.221926997162531 0 rpy=0 0 0 -> xyz=0 -2.0242932765670663 0 rpy=0 0 0
- joint Torso_FrontLowerLeg: origin xyz=0 2.221926997162531 0 rpy=0 0 0 -> xyz=0 2.0242932765670663 0 rpy=0 0 0
- joint Torso_LeftLowerLeg: origin xyz=-1.831290686135426 0 0 rpy=0 0 0 -> xyz=-2.1516290903712636 0 0 rpy=0 0 0
- joint Torso_RightLowerLeg: origin xyz=1.831290686135426 0 0 rpy=0 0 0 -> xyz=2.1516290903712636 0 0 rpy=0 0 0

File: body20.urdf (robot description, URDF)
Before this commit: robot robot, 9 links, 8 joints
Links:
- link BackLeg: geometry collision box size=0.23330725228663526 2.0898445794296574 0.2601007568258945; visual box size=0.23330725228663526 2.0898445794296574 0.2601007568258945
- link BackLowerLeg: geometry collision box size=0.11740774307450663 0.2246331191130643 0.9060855931253461; visual box size=0.11740774307450663 0.2246331191130643 0.9060855931253461
- link FrontLeg: geometry collision box size=0.23330725228663526 2.0898445794296574 0.2601007568258945; visual box size=0.23330725228663526 2.0898445794296574 0.2601007568258945
- link FrontLowerLeg: geometry collision box size=0.11740774307450663 0.2246331191130643 0.9060855931253461; visual box size=0.11740774307450663 0.2246331191130643 0.9060855931253461
- link LeftLeg: geometry collision box size=1.94743209765741 0.21213048905061496 0.10553124110954588; visual box size=1.94743209765741 0.21213048905061496 0.10553124110954588
- link LeftLowerLeg: geometry collision box size=0.15710562601223532 0.29924587877860215 0.8003314228813837; visual box size=0.15710562601223532 0.29924587877860215 0.8003314228813837
- link RightLeg: geometry collision box size=1.94743209765741 0.21213048905061496 0.10553124110954588; visual box size=1.94743209765741 0.21213048905061496 0.10553124110954588
- link RightLowerLeg: geometry collision box size=0.15710562601223532 0.29924587877860215 0.8003314228813837; visual box size=0.15710562601223532 0.29924587877860215 0.8003314228813837
Joints:
- joint Torso_BackLowerLeg: origin xyz=0 -2.0948417418807437 0 rpy=0 0 0 -> xyz=0 -2.0898445794296574 0 rpy=0 0 0
- joint Torso_FrontLowerLeg: origin xyz=0 2.0948417418807437 0 rpy=0 0 0 -> xyz=0 2.0898445794296574 0 rpy=0 0 0
- joint Torso_LeftLowerLeg: origin xyz=-1.845254525118026 0 0 rpy=0 0 0 -> xyz=-1.94743209765741 0 0 rpy=0 0 0
- joint Torso_RightLowerLeg: origin xyz=1.845254525118026 0 0 rpy=0 0 0 -> xyz=1.94743209765741 0 0 rpy=0 0 0

File: body21.urdf (robot description, URDF)
Before this commit: robot robot, 9 links, 8 joints
Links:
- link BackLeg: geometry collision box size=0.1 2.092393832863068 0.23059262525614624; visual box size=0.1 2.092393832863068 0.23059262525614624
- link BackLowerLeg: geometry collision box size=0.32416812713873316 0.1 0.9193885472477775; visual box size=0.32416812713873316 0.1 0.9193885472477775
- link FrontLeg: geometry collision box size=0.1 2.092393832863068 0.23059262525614624; visual box size=0.1 2.092393832863068 0.23059262525614624
- link FrontLowerLeg: geometry collision box size=0.32416812713873316 0.1 0.9193885472477775; visual box size=0.32416812713873316 0.1 0.9193885472477775
- link LeftLeg: geometry collision box size=2.194679663913454 0.12987609344669715 0.3809736315199602; visual box size=2.194679663913454 0.12987609344669715 0.3809736315199602
- link LeftLowerLeg: geometry collision box size=0.24542102716863573 0.1 1.1898114078426927; visual box size=0.24542102716863573 0.1 1.1898114078426927
- link RightLeg: geometry collision box size=2.194679663913454 0.12987609344669715 0.3809736315199602; visual box size=2.194679663913454 0.12987609344669715 0.3809736315199602
- link RightLowerLeg: geometry collision box size=0.24542102716863573 0.1 1.1898114078426927; visual box size=0.24542102716863573 0.1 1.1898114078426927
Joints:
- joint Torso_BackLowerLeg: origin xyz=0 -1.8795610506714615 0 rpy=0 0 0 -> xyz=0 -2.092393832863068 0 rpy=0 0 0
- joint Torso_FrontLowerLeg: origin xyz=0 1.8795610506714615 0 rpy=0 0 0 -> xyz=0 2.092393832863068 0 rpy=0 0 0
- joint Torso_LeftLowerLeg: origin xyz=-1.8055839773827302 0 0 rpy=0 0 0 -> xyz=-2.194679663913454 0 0 rpy=0 0 0
- joint Torso_RightLowerLeg: origin xyz=1.8055839773827302 0 0 rpy=0 0 0 -> xyz=2.194679663913454 0 0 rpy=0 0 0

File: body22.urdf (robot description, URDF)
Before this commit: robot robot, 9 links, 8 joints
Links:
- link BackLeg: geometry collision box size=0.1 2.1098113955523092 0.3386019564368963; visual box size=0.1 2.1098113955523092 0.3386019564368963
- link BackLowerLeg: geometry collision box size=0.38933864070340496 0.1 0.8312294863116384; visual box size=0.38933864070340496 0.1 0.8312294863116384
- link FrontLeg: geometry collision box size=0.1 2.1098113955523092 0.3386019564368963; visual box size=0.1 2.1098113955523092 0.3386019564368963
- link FrontLowerLeg: geometry collision box size=0.38933864070340496 0.1 0.8312294863116384; visual box size=0.38933864070340496 0.1 0.8312294863116384
- link LeftLeg: geometry collision box size=1.9844068633933283 0.2511761668073997 0.27009949956572027; visual box size=1.9844068633933283 0.2511761668073997 0.27009949956572027
- link LeftLowerLeg: geometry collision box size=0.2859617523769417 0.14749525603761168 1.0445882869576741; visual box size=0.2859617523769417 0.14749525603761168 1.0445882869576741
- link RightLeg: geometry collision box size=1.9844068633933283 0.2511761668073997 0.27009949956572027; visual box size=1.9844068633933283 0.2511761668073997 0.27009949956572027
- link RightLowerLeg: geometry collision box size=0.2859617523769417 0.14749525603761168 1.0445882869576741; visual box size=0.2859617523769417 0.14749525603761168 1.0445882869576741
Joints:
- joint Torso_BackLowerLeg: origin xyz=0 -1.9006395926468471 0 rpy=0 0 0 -> xyz=0 -2.1098113955523092 0 rpy=0 0 0
- joint Torso_FrontLowerLeg: origin xyz=0 1.9006395926468471 0 rpy=0 0 0 -> xyz=0 2.1098113955523092 0 rpy=0 0 0
- joint Torso_LeftLowerLeg: origin xyz=-1.9311245312409582 0 0 rpy=0 0 0 -> xyz=-1.9844068633933283 0 0 rpy=0 0 0
- joint Torso_RightLowerLeg: origin xyz=1.9311245312409582 0 0 rpy=0 0 0 -> xyz=1.9844068633933283 0 0 rpy=0 0 0

File: body23.urdf (robot description, URDF)
Before this commit: robot robot, 9 links, 8 joints
Links:
- link BackLeg: geometry collision box size=0.1737933606056049 1.9846098149572695 0.11571989645019674; visual box size=0.1737933606056049 1.9846098149572695 0.11571989645019674
- link BackLowerLeg: geometry collision box size=0.307588700336366 0.1 1.0781640612954229; visual box size=0.307588700336366 0.1 1.0781640612954229
- link FrontLeg: geometry collision box size=0.1737933606056049 1.9846098149572695 0.11571989645019674; visual box size=0.1737933606056049 1.9846098149572695 0.11571989645019674
- link FrontLowerLeg: geometry collision box size=0.307588700336366 0.1 1.0781640612954229; visual box size=0.307588700336366 0.1 1.0781640612954229
- link LeftLeg: geometry collision box size=2.085243857099702 0.1 0.23061900377265843; visual box size=2.085243857099702 0.1 0.23061900377265843
- link LeftLowerLeg: geometry collision box size=0.17173255125169073 0.1 1.1127897719664244; visual box size=0.17173255125169073 0.1 1.1127897719664244
- link RightLeg: geometry collision box size=2.085243857099702 0.1 0.23061900377265843; visual box size=2.085243857099702 0.1 0.23061900377265843
- link RightLowerLeg: geometry collision box size=0.17173255125169073 0.1 1.1127897719664244; visual box size=0.17173255125169073 0.1 1.1127897719664244
Joints:
- joint Torso_BackLowerLeg: origin xyz=0 -2.177081201168779 0 rpy=0 0 0 -> xyz=0 -1.9846098149572695 0 rpy=0 0 0
- joint Torso_FrontLowerLeg: origin xyz=0 2.177081201168779 0 rpy=0 0 0 -> xyz=0 1.9846098149572695 0 rpy=0 0 0
- joint Torso_LeftLowerLeg: origin xyz=-2.0083836864552107 0 0 rpy=0 0 0 -> xyz=-2.085243857099702 0 0 rpy=0 0 0
- joint Torso_RightLowerLeg: origin xyz=2.0083836864552107 0 0 rpy=0 0 0 -> xyz=2.085243857099702 0 0 rpy=0 0 0
