Commit message: milestone 4 done

File: body24.urdf (robot description, URDF)
Before this commit: robot robot, 9 links, 8 joints
Links:
- link BackLeg: geometry collision box size=0.160174455902762 1.8943071083175564 0.3890015619741935; visual box size=0.160174455902762 1.8943071083175564 0.3890015619741935
- link BackLowerLeg: geometry collision box size=0.1 0.15735961587905511 1.1272893559593724; visual box size=0.1 0.15735961587905511 1.1272893559593724
- link FrontLeg: geometry collision box size=0.160174455902762 1.8943071083175564 0.3890015619741935; visual box size=0.160174455902762 1.8943071083175564 0.3890015619741935
- link FrontLowerLeg: geometry collision box size=0.1 0.15735961587905511 1.1272893559593724; visual box size=0.1 0.15735961587905511 1.1272893559593724
- link LeftLeg: geometry collision box size=1.9010885943221014 0.37561095085189056 0.18565322229522474; visual box size=1.9010885943221014 0.37561095085189056 0.18565322229522474
- link LeftLowerLeg: geometry collision box size=0.1 0.14855432448626724 0.8865446102125144; visual box size=0.1 0.14855432448626724 0.8865446102125144
- link RightLeg: geometry collision box size=1.9010885943221014 0.37561095085189056 0.18565322229522474; visual box size=1.9010885943221014 0.37561095085189056 0.18565322229522474
- link RightLowerLeg: geometry collision box size=0.1 0.14855432448626724 0.8865446102125144; visual box size=0.1 0.14855432448626724 0.8865446102125144
Joints:
- joint Torso_BackLowerLeg: origin xyz=0 -2.19972151574263 0 rpy=0 0 0 -> xyz=0 -1.8943071083175564 0 rpy=0 0 0
- joint Torso_FrontLowerLeg: origin xyz=0 2.19972151574263 0 rpy=0 0 0 -> xyz=0 1.8943071083175564 0 rpy=0 0 0
- joint Torso_LeftLowerLeg: origin xyz=-2.024105548797988 0 0 rpy=0 0 0 -> xyz=-1.9010885943221014 0 0 rpy=0 0 0
- joint Torso_RightLowerLeg: origin xyz=2.024105548797988 0 0 rpy=0 0 0 -> xyz=1.9010885943221014 0 0 rpy=0 0 0

File: body25.urdf (robot description, URDF)
Before this commit: robot robot, 9 links, 8 joints
Links:
- link BackLeg: geometry collision box size=0.39612988569357854 2.183448960088439 0.3997370420629495; visual box size=0.39612988569357854 2.183448960088439 0.3997370420629495
- link BackLowerLeg: geometry collision box size=0.3112373220003424 0.39248906125083144 0.9778606678133157; visual box size=0.3112373220003424 0.39248906125083144 0.9778606678133157
- link FrontLeg: geometry collision box size=0.39612988569357854 2.183448960088439 0.3997370420629495; visual box size=0.39612988569357854 2.183448960088439 0.3997370420629495
- link FrontLowerLeg: geometry collision box size=0.3112373220003424 0.39248906125083144 0.9778606678133157; visual box size=0.3112373220003424 0.39248906125083144 0.9778606678133157
- link LeftLeg: geometry collision box size=2.0524636876978666 0.1 0.2802816363339586; visual box size=2.0524636876978666 0.1 0.2802816363339586
- link LeftLowerLeg: geometry collision box size=0.3623969711448996 0.17981969022781033 1.1517173724106193; visual box size=0.3623969711448996 0.17981969022781033 1.1517173724106193
- link RightLeg: geometry collision box size=2.0524636876978666 0.1 0.2802816363339586; visual box size=2.0524636876978666 0.1 0.2802816363339586
- link RightLowerLeg: geometry collision box size=0.3623969711448996 0.17981969022781033 1.1517173724106193; visual box size=0.3623969711448996 0.17981969022781033 1.1517173724106193
Joints:
- joint Torso_BackLowerLeg: origin xyz=0 -1.9769062200278906 0 rpy=0 0 0 -> xyz=0 -2.183448960088439 0 rpy=0 0 0
- joint Torso_FrontLowerLeg: origin xyz=0 1.9769062200278906 0 rpy=0 0 0 -> xyz=0 2.183448960088439 0 rpy=0 0 0
- joint Torso_LeftLowerLeg: origin xyz=-1.952052715475317 0 0 rpy=0 0 0 -> xyz=-2.0524636876978666 0 0 rpy=0 0 0
- joint Torso_RightLowerLeg: origin xyz=1.952052715475317 0 0 rpy=0 0 0 -> xyz=2.0524636876978666 0 0 rpy=0 0 0

File: body26.urdf (robot description, URDF)
Before this commit: robot robot, 9 links, 8 joints
Links:
- link BackLeg: geometry collision box size=0.3920565734922725 1.9891449096967302 0.3494230603385682; visual box size=0.3920565734922725 1.9891449096967302 0.3494230603385682
- link BackLowerLeg: geometry collision box size=0.1 0.39374639837348596 0.8639012966486029; visual box size=0.1 0.39374639837348596 0.8639012966486029
- link FrontLeg: geometry collision box size=0.3920565734922725 1.9891449096967302 0.3494230603385682; visual box size=0.3920565734922725 1.9891449096967302 0.3494230603385682
- link FrontLowerLeg: geometry collision box size=0.1 0.39374639837348596 0.8639012966486029; visual box size=0.1 0.39374639837348596 0.8639012966486029
- link LeftLeg: geometry collision box size=2.1258569105031833 0.20434552856162957 0.3285535629853088; visual box size=2.1258569105031833 0.20434552856162957 0.3285535629853088
- link LeftLowerLeg: geometry collision box size=0.35286514963699656 0.28523779771824154 0.9368929223534096; visual box size=0.35286514963699656 0.28523779771824154 0.9368929223534096
- link RightLeg: geometry collision box size=2.1258569105031833 0.20434552856162957 0.3285535629853088; visual box size=2.1258569105031833 0.20434552856162957 0.3285535629853088
- link RightLowerLeg: geometry collision box size=0.35286514963699656 0.28523779771824154 0.9368929223534096; visual box size=0.35286514963699656 0.28523779771824154 0.9368929223534096
Joints:
- joint Torso_BackLowerLeg: origin xyz=0 -2.083439347529 0 rpy=0 0 0 -> xyz=0 -1.9891449096967302 0 rpy=0 0 0
- joint Torso_FrontLowerLeg: origin xyz=0 2.083439347529 0 rpy=0 0 0 -> xyz=0 1.9891449096967302 0 rpy=0 0 0
- joint Torso_LeftLowerLeg: origin xyz=-1.814803256340219 0 0 rpy=0 0 0 -> xyz=-2.1258569105031833 0 0 rpy=0 0 0
- joint Torso_RightLowerLeg: origin xyz=1.814803256340219 0 0 rpy=0 0 0 -> xyz=2.1258569105031833 0 0 rpy=0 0 0

File: body27.urdf (robot description, URDF)
Before this commit: robot robot, 9 links, 8 joints
Links:
- link BackLeg: geometry collision box size=0.16294009176770352 1.8079597080002516 0.300048186228994; visual box size=0.16294009176770352 1.8079597080002516 0.300048186228994
- link BackLowerLeg: geometry collision box size=0.1 0.1892824429230529 0.9077571330214806; visual box size=0.1 0.1892824429230529 0.9077571330214806
- link FrontLeg: geometry collision box size=0.16294009176770352 1.8079597080002516 0.300048186228994; visual box size=0.16294009176770352 1.8079597080002516 0.300048186228994
- link FrontLowerLeg: geometry collision box size=0.1 0.1892824429230529 0.9077571330214806; visual box size=0.1 0.1892824429230529 0.9077571330214806
- link LeftLeg: geometry collision box size=2.115811106999617 0.28867026403550716 0.17237619623414108; visual box size=2.115811106999617 0.28867026403550716 0.17237619623414108
- link LeftLowerLeg: geometry collision box size=0.1 0.170163564207591 1.1085181957781458; visual box size=0.1 0.170163564207591 1.1085181957781458
- link RightLeg: geometry collision box size=2.115811106999617 0.28867026403550716 0.17237619623414108; visual box size=2.115811106999617 0.28867026403550716 0.17237619623414108
- link RightLowerLeg: geometry collision box size=0.1 0.170163564207591 1.1085181957781458; visual box size=0.1 0.170163564207591 1.1085181957781458
Joints:
- joint Torso_BackLowerLeg: origin xyz=0 -1.8470312269087545 0 rpy=0 0 0 -> xyz=0 -1.8079597080002516 0 rpy=0 0 0
- joint Torso_FrontLowerLeg: origin xyz=0 1.8470312269087545 0 rpy=0 0 0 -> xyz=0 1.8079597080002516 0 rpy=0 0 0
- joint Torso_LeftLowerLeg: origin xyz=-1.917229370844435 0 0 rpy=0 0 0 -> xyz=-2.115811106999617 0 0 rpy=0 0 0
- joint Torso_RightLowerLeg: origin xyz=1.917229370844435 0 0 rpy=0 0 0 -> xyz=2.115811106999617 0 0 rpy=0 0 0

File: body28.urdf (robot description, URDF)
Before this commit: robot robot, 9 links, 8 joints
Links:
- link BackLeg: geometry collision box size=0.2944236504813605 1.9184989659322975 0.2488903313475075; visual box size=0.2944236504813605 1.9184989659322975 0.2488903313475075
- link BackLowerLeg: geometry collision box size=0.1 0.37694015009649817 1.1840913210513955; visual box size=0.1 0.37694015009649817 1.1840913210513955
- link FrontLeg: geometry collision box size=0.2944236504813605 1.9184989659322975 0.2488903313475075; visual box size=0.2944236504813605 1.9184989659322975 0.2488903313475075
- link FrontLowerLeg: geometry collision box size=0.1 0.37694015009649817 1.1840913210513955; visual box size=0.1 0.37694015009649817 1.1840913210513955
- link LeftLeg: geometry collision box size=2.194876995655079 0.29211394806316 0.260193500678131; visual box size=2.194876995655079 0.29211394806316 0.260193500678131
- link LeftLowerLeg: geometry collision box size=0.1 0.3782392949475872 1.1573615413439833; visual box size=0.1 0.3782392949475872 1.1573615413439833
- link RightLeg: geometry collision box size=2.194876995655079 0.29211394806316 0.260193500678131; visual box size=2.194876995655079 0.29211394806316 0.260193500678131
- link RightLowerLeg: geometry collision box size=0.1 0.3782392949475872 1.1573615413439833; visual box size=0.1 0.3782392949475872 1.1573615413439833
Joints:
- joint Torso_BackLowerLeg: origin xyz=0 -2.091513519679978 0 rpy=0 0 0 -> xyz=0 -1.9184989659322975 0 rpy=0 0 0
- joint Torso_FrontLowerLeg: origin xyz=0 2.091513519679978 0 rpy=0 0 0 -> xyz=0 1.9184989659322975 0 rpy=0 0 0
- joint Torso_LeftLowerLeg: origin xyz=-1.8397547740281959 0 0 rpy=0 0 0 -> xyz=-2.194876995655079 0 0 rpy=0 0 0
- joint Torso_RightLowerLeg: origin xyz=1.8397547740281959 0 0 rpy=0 0 0 -> xyz=2.194876995655079 0 0 rpy=0 0 0

File: body29.urdf (robot description, URDF)
Before this commit: robot robot, 9 links, 8 joints
Links:
- link BackLeg: geometry collision box size=0.38098871756495806 2.0721219701351106 0.10259844644868266; visual box size=0.38098871756495806 2.0721219701351106 0.10259844644868266
- link BackLowerLeg: geometry collision box size=0.14173362645630055 0.1 0.9846742328491327; visual box size=0.14173362645630055 0.1 0.9846742328491327
- link FrontLeg: geometry collision box size=0.38098871756495806 2.0721219701351106 0.10259844644868266; visual box size=0.38098871756495806 2.0721219701351106 0.10259844644868266
- link FrontLowerLeg: geometry collision box size=0.14173362645630055 0.1 0.9846742328491327; visual box size=0.14173362645630055 0.1 0.9846742328491327
- link LeftLeg: geometry collision box size=2.165410495993395 0.16929100046570925 0.33939240345723787; visual box size=2.165410495993395 0.16929100046570925 0.33939240345723787
- link LeftLowerLeg: geometry collision box size=0.10409174365229196 0.1916813581789099 0.9427686157629467; visual box size=0.10409174365229196 0.1916813581789099 0.9427686157629467
- link RightLeg: geometry collision box size=2.165410495993395 0.16929100046570925 0.33939240345723787; visual box size=2.165410495993395 0.16929100046570925 0.33939240345723787
- link RightLowerLeg: geometry collision box size=0.10409174365229196 0.1916813581789099 0.9427686157629467; visual box size=0.10409174365229196 0.1916813581789099 0.9427686157629467
Joints:
- joint Torso_BackLowerLeg: origin xyz=0 -2.0872385847077206 0 rpy=0 0 0 -> xyz=0 -2.0721219701351106 0 rpy=0 0 0
- joint Torso_FrontLowerLeg: origin xyz=0 2.0872385847077206 0 rpy=0 0 0 -> xyz=0 2.0721219701351106 0 rpy=0 0 0
- joint Torso_LeftLowerLeg: origin xyz=-1.9450566545074963 0 0 rpy=0 0 0 -> xyz=-2.165410495993395 0 0 rpy=0 0 0
- joint Torso_RightLowerLeg: origin xyz=1.9450566545074963 0 0 rpy=0 0 0 -> xyz=2.165410495993395 0 0 rpy=0 0 0
