Commit message: For loop that goes through both symmetric and non symmetric and then graphs them both

File: body100.urdf (robot description, URDF)
Before this commit: robot robot, 9 links, 8 joints
Links:
- link BackLeg: geometry collision box size=0.32505783075593186 2.0116093912968154 0.13301298747587623; visual box size=0.32505783075593186 2.0116093912968154 0.13301298747587623
- link BackLowerLeg: geometry collision box size=0.1 0.2822239422375915 0.94088798136795; visual box size=0.1 0.2822239422375915 0.94088798136795
- link FrontLeg: geometry collision box size=0.3780649247269704 2.1117779375669974 0.1; visual box size=0.3780649247269704 2.1117779375669974 0.1
- link FrontLowerLeg: geometry collision box size=0.3276599676554677 0.20141695677248808 1.1083802742200173; visual box size=0.3276599676554677 0.20141695677248808 1.1083802742200173
- link LeftLeg: geometry collision box size=1.8798969393669138 0.3846149173565281 0.3823081277351055; visual box size=1.8798969393669138 0.3846149173565281 0.3823081277351055
- link LeftLowerLeg: geometry collision box size=0.19717545090088073 0.20434831282801477 0.861955362023759; visual box size=0.19717545090088073 0.20434831282801477 0.861955362023759
- link RightLeg: geometry collision box size=1.949407073601662 0.1 0.10106153148940106; visual box size=1.949407073601662 0.1 0.10106153148940106
- link RightLowerLeg: geometry collision box size=0.39184779402068315 0.12587230127211774 0.8429415117406711; visual box size=0.39184779402068315 0.12587230127211774 0.8429415117406711
Joints:
- joint Torso_BackLowerLeg: origin xyz=0 -1.9951351016371128 0 rpy=0 0 0 -> xyz=0 -2.0116093912968154 0 rpy=0 0 0
- joint Torso_FrontLowerLeg: origin xyz=0 1.9951351016371128 0 rpy=0 0 0 -> xyz=0 2.1117779375669974 0 rpy=0 0 0
- joint Torso_LeftLowerLeg: origin xyz=-2.0989685176853774 0 0 rpy=0 0 0 -> xyz=-1.8798969393669138 0 0 rpy=0 0 0
- joint Torso_RightLowerLeg: origin xyz=2.0989685176853774 0 0 rpy=0 0 0 -> xyz=1.949407073601662 0 0 rpy=0 0 0

File: body1000.urdf (robot description, URDF)
Before this commit: robot robot, 9 links, 8 joints
Links:
- link BackLeg: geometry collision box size=0.24113206501840825 1.6458032112048573 0.22888941012153916; visual box size=0.24113206501840825 1.6458032112048573 0.22888941012153916
- link BackLowerLeg: geometry collision box size=0.5912674953704362 0.13077387788272848 1.1436085040505748; visual box size=0.5912674953704362 0.13077387788272848 1.1436085040505748
- link FrontLeg: geometry collision box size=0.630150414892046 2.0067565367307245 0.5996854788450767; visual box size=0.630150414892046 2.0067565367307245 0.5996854788450767
- link FrontLowerLeg: geometry collision box size=0.22573541721463936 0.4107370102571811 1.0722926333349156; visual box size=0.22573541721463936 0.4107370102571811 1.0722926333349156
- link LeftLeg: geometry collision box size=1.4530373838094972 0.1 0.5588018607584724; visual box size=1.4530373838094972 0.1 0.5588018607584724
- link LeftLowerLeg: geometry collision box size=0.29944994485354326 0.1 0.9128941241674406; visual box size=0.29944994485354326 0.1 0.9128941241674406
- link RightLeg: geometry collision box size=1.904517721832468 0.1 0.1; visual box size=1.904517721832468 0.1 0.1
- link RightLowerLeg: geometry collision box size=0.3139898562587527 0.1 0.8891023806290399; visual box size=0.3139898562587527 0.1 0.8891023806290399
Joints:
- joint Torso_BackLowerLeg: origin xyz=0 -2.0699310739097774 0 rpy=0 0 0 -> xyz=0 -1.6458032112048573 0 rpy=0 0 0
- joint Torso_FrontLowerLeg: origin xyz=0 2.0699310739097774 0 rpy=0 0 0 -> xyz=0 2.0067565367307245 0 rpy=0 0 0
- joint Torso_LeftLowerLeg: origin xyz=-2.0889425202022274 0 0 rpy=0 0 0 -> xyz=-1.4530373838094972 0 0 rpy=0 0 0
- joint Torso_RightLowerLeg: origin xyz=2.0889425202022274 0 0 rpy=0 0 0 -> xyz=1.904517721832468 0 0 rpy=0 0 0

File: body1001.urdf (robot description, URDF)
Before this commit: robot robot, 9 links, 8 joints
Links:
- link BackLeg: geometry collision box size=0.47132705349006887 2.1269368563085793 0.4502567451505506; visual box size=0.47132705349006887 2.1269368563085793 0.4502567451505506
- link BackLowerLeg: geometry collision box size=0.33213920754753423 0.7039073544564106 1.5278349098074073; visual box size=0.33213920754753423 0.7039073544564106 1.5278349098074073
- link FrontLeg: geometry collision box size=0.3196394009243202 1.4789507235478176 0.16431903430879094; visual box size=0.3196394009243202 1.4789507235478176 0.16431903430879094
- link FrontLowerLeg: geometry collision box size=0.2696823126160546 0.22263031357386154 1.4219979780117264; visual box size=0.2696823126160546 0.22263031357386154 1.4219979780117264
- link LeftLeg: geometry collision box size=2.309502534104664 0.1 0.6411985816569271; visual box size=2.309502534104664 0.1 0.6411985816569271
- link LeftLowerLeg: geometry collision box size=0.10985821139116131 0.28475053342899587 1.2905056285610557; visual box size=0.10985821139116131 0.28475053342899587 1.2905056285610557
- link RightLeg: geometry collision box size=1.2875186097451778 0.5068613810640876 0.1560287788407344; visual box size=1.2875186097451778 0.5068613810640876 0.1560287788407344
- link RightLowerLeg: geometry collision box size=0.5749595632027674 0.6197824005396846 1.7374251796594393; visual box size=0.5749595632027674 0.6197824005396846 1.7374251796594393
Joints:
- joint Torso_BackLowerLeg: origin xyz=0 -2.44177702030001 0 rpy=0 0 0 -> xyz=0 -2.1269368563085793 0 rpy=0 0 0
- joint Torso_FrontLowerLeg: origin xyz=0 2.44177702030001 0 rpy=0 0 0 -> xyz=0 1.4789507235478176 0 rpy=0 0 0
- joint Torso_LeftLowerLeg: origin xyz=-2.195970254064227 0 0 rpy=0 0 0 -> xyz=-2.309502534104664 0 0 rpy=0 0 0
- joint Torso_RightLowerLeg: origin xyz=2.195970254064227 0 0 rpy=0 0 0 -> xyz=1.2875186097451778 0 0 rpy=0 0 0

File: body1002.urdf (robot description, URDF)
Before this commit: robot robot, 9 links, 8 joints
Links:
- link BackLeg: geometry collision box size=0.4306002154439978 0.7403529238243094 0.3121851995279006; visual box size=0.4306002154439978 0.7403529238243094 0.3121851995279006
- link BackLowerLeg: geometry collision box size=0.16686858229113885 0.5191691020715485 0.6490359228074779; visual box size=0.16686858229113885 0.5191691020715485 0.6490359228074779
- link FrontLeg: geometry collision box size=0.37349265432789336 2.247445226268682 0.6270725671828044; visual box size=0.37349265432789336 2.247445226268682 0.6270725671828044
- link FrontLowerLeg: geometry collision box size=0.1 0.1 1.3572271027807155; visual box size=0.1 0.1 1.3572271027807155
- link LeftLeg: geometry collision box size=1.817500450633569 0.1 0.1761025072854974; visual box size=1.817500450633569 0.1 0.1761025072854974
- link LeftLowerLeg: geometry collision box size=0.26738172360429324 0.1 1.0595015767788103; visual box size=0.26738172360429324 0.1 1.0595015767788103
- link RightLeg: geometry collision box size=1.862974828596033 0.49574464282737263 0.35878669202985514; visual box size=1.862974828596033 0.49574464282737263 0.35878669202985514
- link RightLowerLeg: geometry collision box size=1.2964666675384071 1.0896339170904137 1.642413837894271; visual box size=1.2964666675384071 1.0896339170904137 1.642413837894271
Joints:
- joint Torso_BackLowerLeg: origin xyz=0 -1.9779378945020718 0 rpy=0 0 0 -> xyz=0 -0.7403529238243094 0 rpy=0 0 0
- joint Torso_FrontLowerLeg: origin xyz=0 1.9779378945020718 0 rpy=0 0 0 -> xyz=0 2.247445226268682 0 rpy=0 0 0
- joint Torso_LeftLowerLeg: origin xyz=-2.026239783915447 0 0 rpy=0 0 0 -> xyz=-1.817500450633569 0 0 rpy=0 0 0
- joint Torso_RightLowerLeg: origin xyz=2.026239783915447 0 0 rpy=0 0 0 -> xyz=1.862974828596033 0 0 rpy=0 0 0

File: body1003.urdf (robot description, URDF)
Before this commit: robot robot, 9 links, 8 joints
Links:
- link BackLeg: geometry collision box size=0.3912154975159662 2.504164523039834 1.125228944266405; visual box size=0.3912154975159662 2.504164523039834 1.125228944266405
- link BackLowerLeg: geometry collision box size=0.3135628748605357 0.9471808577087821 0.9471285926519691; visual box size=0.3135628748605357 0.9471808577087821 0.9471285926519691
- link FrontLeg: geometry collision box size=0.10838991577877866 2.2600657456417568 0.3552603274367908; visual box size=0.10838991577877866 2.2600657456417568 0.3552603274367908
- link FrontLowerLeg: geometry collision box size=0.2665521401518459 0.1 1.2077878789829901; visual box size=0.2665521401518459 0.1 1.2077878789829901
- link LeftLeg: geometry collision box size=2.0403402378034405 0.5515758818375383 0.25389569824700287; visual box size=2.0403402378034405 0.5515758818375383 0.25389569824700287
- link LeftLowerLeg: geometry collision box size=0.2179533095703503 0.4414974415707769 0.15979730782215562; visual box size=0.2179533095703503 0.4414974415707769 0.15979730782215562
- link RightLeg: geometry collision box size=2.0944142344959094 0.6710126404365339 0.28401127590127695; visual box size=2.0944142344959094 0.6710126404365339 0.28401127590127695
- link RightLowerLeg: geometry collision box size=0.5229854831293952 0.3764430532734239 1.21865542460311; visual box size=0.5229854831293952 0.3764430532734239 1.21865542460311
Joints:
- joint Torso_BackLowerLeg: origin xyz=0 -1.668707709365941 0 rpy=0 0 0 -> xyz=0 -2.504164523039834 0 rpy=0 0 0
- joint Torso_FrontLowerLeg: origin xyz=0 1.668707709365941 0 rpy=0 0 0 -> xyz=0 2.2600657456417568 0 rpy=0 0 0
- joint Torso_LeftLowerLeg: origin xyz=-1.8612293202212558 0 0 rpy=0 0 0 -> xyz=-2.0403402378034405 0 0 rpy=0 0 0
- joint Torso_RightLowerLeg: origin xyz=1.8612293202212558 0 0 rpy=0 0 0 -> xyz=2.0944142344959094 0 0 rpy=0 0 0

File: body1004.urdf (robot description, URDF)
Before this commit: robot robot, 9 links, 8 joints
Links:
- link BackLeg: geometry collision box size=0.1 2.2934145632290406 0.6890742768757698; visual box size=0.1 2.2934145632290406 0.6890742768757698
- link BackLowerLeg: geometry collision box size=0.32850126334559937 0.9116237240369589 1.0390475706215403; visual box size=0.32850126334559937 0.9116237240369589 1.0390475706215403
- link FrontLeg: geometry collision box size=0.4654456945954542 1.7599183954104713 0.5337884217107551; visual box size=0.4654456945954542 1.7599183954104713 0.5337884217107551
- link FrontLowerLeg: geometry collision box size=0.55780193021476 0.4393426940472168 1.563817167277744; visual box size=0.55780193021476 0.4393426940472168 1.563817167277744
- link LeftLeg: geometry collision box size=1.3893968986095233 0.40277599839818523 0.13029113731929562; visual box size=1.3893968986095233 0.40277599839818523 0.13029113731929562
- link LeftLowerLeg: geometry collision box size=0.15306259401195854 0.41007051223801994 1.2431733644299916; visual box size=0.15306259401195854 0.41007051223801994 1.2431733644299916
- link RightLeg: geometry collision box size=1.6583599491659522 0.1 0.7658100704968493; visual box size=1.6583599491659522 0.1 0.7658100704968493
- link RightLowerLeg: geometry collision box size=0.11367887601950843 0.6013013695157646 1.4439739593856016; visual box size=0.11367887601950843 0.6013013695157646 1.4439739593856016
Joints:
- joint Torso_BackLowerLeg: origin xyz=0 -2.15436128875035 0 rpy=0 0 0 -> xyz=0 -2.2934145632290406 0 rpy=0 0 0
- joint Torso_FrontLowerLeg: origin xyz=0 2.15436128875035 0 rpy=0 0 0 -> xyz=0 1.7599183954104713 0 rpy=0 0 0
- joint Torso_LeftLowerLeg: origin xyz=-2.4005415416551563 0 0 rpy=0 0 0 -> xyz=-1.3893968986095233 0 0 rpy=0 0 0
- joint Torso_RightLowerLeg: origin xyz=2.4005415416551563 0 0 rpy=0 0 0 -> xyz=1.6583599491659522 0 0 rpy=0 0 0

File: body1005.urdf (robot description, URDF)
Before this commit: robot robot, 9 links, 8 joints
Links:
- link BackLeg: geometry collision box size=0.28923545629270814 2.084113447863887 0.28386922652390845; visual box size=0.28923545629270814 2.084113447863887 0.28386922652390845
- link BackLowerLeg: geometry collision box size=0.5338228413673202 0.1 1.4917497554899066; visual box size=0.5338228413673202 0.1 1.4917497554899066
- link FrontLeg: geometry collision box size=0.5117294242942765 2.0877476856217556 0.7056073247530795; visual box size=0.5117294242942765 2.0877476856217556 0.7056073247530795
- link FrontLowerLeg: geometry collision box size=0.6581991154300967 0.22151237394563095 1.1750319603618975; visual box size=0.6581991154300967 0.22151237394563095 1.1750319603618975
- link LeftLeg: geometry collision box size=2.429053131893011 0.6932298528095697 0.33842507231026075; visual box size=2.429053131893011 0.6932298528095697 0.33842507231026075
- link LeftLowerLeg: geometry collision box size=0.1 0.10364142191578388 0.5030245822062605; visual box size=0.1 0.10364142191578388 0.5030245822062605
- link RightLeg: geometry collision box size=2.0345500499778857 0.17860684396513038 0.3676093251193313; visual box size=2.0345500499778857 0.17860684396513038 0.3676093251193313
- link RightLowerLeg: geometry collision box size=0.3839232512301722 0.4232618946297787 1.263987749360842; visual box size=0.3839232512301722 0.4232618946297787 1.263987749360842
Joints:
- joint Torso_BackLowerLeg: origin xyz=0 -2.374649188778479 0 rpy=0 0 0 -> xyz=0 -2.084113447863887 0 rpy=0 0 0
- joint Torso_FrontLowerLeg: origin xyz=0 2.374649188778479 0 rpy=0 0 0 -> xyz=0 2.0877476856217556 0 rpy=0 0 0
- joint Torso_LeftLowerLeg: origin xyz=-2.0972279067159927 0 0 rpy=0 0 0 -> xyz=-2.429053131893011 0 0 rpy=0 0 0
- joint Torso_RightLowerLeg: origin xyz=2.0972279067159927 0 0 rpy=0 0 0 -> xyz=2.0345500499778857 0 0 rpy=0 0 0

File: body1006.urdf (robot description, URDF)
Before this commit: robot robot, 9 links, 8 joints
Links:
- link BackLeg: geometry collision box size=0.5716190071727901 2.2147367826611006 0.7473723748989433; visual box size=0.5716190071727901 2.2147367826611006 0.7473723748989433
- link BackLowerLeg: geometry collision box size=0.19779448986049117 0.17936372473729031 1.1274730423941755; visual box size=0.19779448986049117 0.17936372473729031 1.1274730423941755
- link FrontLeg: geometry collision box size=0.1563746114419035 2.0216637631723486 0.27098644644648906; visual box size=0.1563746114419035 2.0216637631723486 0.27098644644648906
- link FrontLowerLeg: geometry collision box size=0.14884580996436345 0.5703838776377556 0.969939857695044; visual box size=0.14884580996436345 0.5703838776377556 0.969939857695044
- link LeftLeg: geometry collision box size=2.36137727236097 0.4871141440287187 0.15713946083575722; visual box size=2.36137727236097 0.4871141440287187 0.15713946083575722
- link LeftLowerLeg: geometry collision box size=0.5364531580926042 0.1420302928684739 1.095947953102315; visual box size=0.5364531580926042 0.1420302928684739 1.095947953102315
- link RightLeg: geometry collision box size=2.3462909565603822 0.1 0.4900731670124991; visual box size=2.3462909565603822 0.1 0.4900731670124991
- link RightLowerLeg: geometry collision box size=0.1 0.2767693483148419 1.2702838664985396; visual box size=0.1 0.2767693483148419 1.2702838664985396
Joints:
- joint Torso_BackLowerLeg: origin xyz=0 -1.6486860327058503 0 rpy=0 0 0 -> xyz=0 -2.2147367826611006 0 rpy=0 0 0
- joint Torso_FrontLowerLeg: origin xyz=0 1.6486860327058503 0 rpy=0 0 0 -> xyz=0 2.0216637631723486 0 rpy=0 0 0
- joint Torso_LeftLowerLeg: origin xyz=-2.184584858505139 0 0 rpy=0 0 0 -> xyz=-2.36137727236097 0 0 rpy=0 0 0
- joint Torso_RightLowerLeg: origin xyz=2.184584858505139 0 0 rpy=0 0 0 -> xyz=2.3462909565603822 0 0 rpy=0 0 0

File: body1007.urdf (robot description, URDF)
Before this commit: robot robot, 9 links, 8 joints
Links:
- link BackLeg: geometry collision box size=0.1 2.206853884876059 0.2586741655081971; visual box size=0.1 2.206853884876059 0.2586741655081971
- link BackLowerLeg: geometry collision box size=0.22588989505073595 0.2968990840040541 0.754083032723436; visual box size=0.22588989505073595 0.2968990840040541 0.754083032723436
- link FrontLeg: geometry collision box size=0.3939349967042557 2.0307646227626686 0.40873655796925645; visual box size=0.3939349967042557 2.0307646227626686 0.40873655796925645
- link FrontLowerLeg: geometry collision box size=0.5625393104766682 0.1 0.9833872658115796; visual box size=0.5625393104766682 0.1 0.9833872658115796
- link LeftLeg: geometry collision box size=2.3020450016481853 0.658276644191265 0.8589624181541519; visual box size=2.3020450016481853 0.658276644191265 0.8589624181541519
- link LeftLowerLeg: geometry collision box size=0.19886090818747398 0.46186532536711555 0.4135114791180642; visual box size=0.19886090818747398 0.46186532536711555 0.4135114791180642
- link RightLeg: geometry collision box size=1.9167333998803144 0.1 0.1; visual box size=1.9167333998803144 0.1 0.1
- link RightLowerLeg: geometry collision box size=0.2707689001187037 0.37786544586029974 1.4446022597534294; visual box size=0.2707689001187037 0.37786544586029974 1.4446022597534294
Joints:
- joint Torso_BackLowerLeg: origin xyz=0 -1.9525707744259468 0 rpy=0 0 0 -> xyz=0 -2.206853884876059 0 rpy=0 0 0
- joint Torso_FrontLowerLeg: origin xyz=0 1.9525707744259468 0 rpy=0 0 0 -> xyz=0 2.0307646227626686 0 rpy=0 0 0
- joint Torso_LeftLowerLeg: origin xyz=-1.9659643425610125 0 0 rpy=0 0 0 -> xyz=-2.3020450016481853 0 0 rpy=0 0 0
- joint Torso_RightLowerLeg: origin xyz=1.9659643425610125 0 0 rpy=0 0 0 -> xyz=1.9167333998803144 0 0 rpy=0 0 0

File: body1008.urdf (robot description, URDF)
Before this commit: robot robot, 9 links, 8 joints
Links:
- link BackLeg: geometry collision box size=0.5652632148196197 1.838672926741358 0.33315089811301724; visual box size=0.5652632148196197 1.838672926741358 0.33315089811301724
- link BackLowerLeg: geometry collision box size=0.6381705616600561 0.1 0.882909880964881; visual box size=0.6381705616600561 0.1 0.882909880964881
- link FrontLeg: geometry collision box size=0.3347596156738825 1.8418714539570793 0.3827242153491994; visual box size=0.3347596156738825 1.8418714539570793 0.3827242153491994
- link FrontLowerLeg: geometry collision box size=0.2868637420972143 0.1 0.8830874919526759; visual box size=0.2868637420972143 0.1 0.8830874919526759
- link LeftLeg: geometry collision box size=1.7661968203553362 0.1 0.11994261429334455; visual box size=1.7661968203553362 0.1 0.11994261429334455
- link LeftLowerLeg: geometry collision box size=0.332626577660286 0.2234256351974769 1.1030143105743586; visual box size=0.332626577660286 0.2234256351974769 1.1030143105743586
- link RightLeg: geometry collision box size=2.0904366344565215 0.3076367260077082 0.1; visual box size=2.0904366344565215 0.3076367260077082 0.1
- link RightLowerLeg: geometry collision box size=0.6561761885096398 0.26246472604922966 0.9547327067981222; visual box size=0.6561761885096398 0.26246472604922966 0.9547327067981222
Joints:
- joint Torso_BackLowerLeg: origin xyz=0 -2.252904873279387 0 rpy=0 0 0 -> xyz=0 -1.838672926741358 0 rpy=0 0 0
- joint Torso_FrontLowerLeg: origin xyz=0 2.252904873279387 0 rpy=0 0 0 -> xyz=0 1.8418714539570793 0 rpy=0 0 0
- joint Torso_LeftLowerLeg: origin xyz=-1.6526246895727073 0 0 rpy=0 0 0 -> xyz=-1.7661968203553362 0 0 rpy=0 0 0
- joint Torso_RightLowerLeg: origin xyz=1.6526246895727073 0 0 rpy=0 0 0 -> xyz=2.0904366344565215 0 0 rpy=0 0 0

File: body1009.urdf (robot description, URDF)
Before this commit: robot robot, 9 links, 8 joints
Links:
- link BackLeg: geometry collision box size=0.3731042884596927 1.7085554522910011 0.1; visual box size=0.3731042884596927 1.7085554522910011 0.1
- link BackLowerLeg: geometry collision box size=0.10044077398597925 0.17391788073874795 0.9488194383630606; visual box size=0.10044077398597925 0.17391788073874795 0.9488194383630606
- link FrontLeg: geometry collision box size=0.3780621241388936 1.5157268514727786 0.34523204897296944; visual box size=0.3780621241388936 1.5157268514727786 0.34523204897296944
- link FrontLowerLeg: geometry collision box size=1.0063756327373232 0.5449201258050149 0.6305120883335179; visual box size=1.0063756327373232 0.5449201258050149 0.6305120883335179
- link LeftLeg: geometry collision box size=2.1483153574910983 0.47552448722375096 0.4062030960228238; visual box size=2.1483153574910983 0.47552448722375096 0.4062030960228238
- link LeftLowerLeg: geometry collision box size=0.20569473673343697 0.603184882797648 0.6797492006351037; visual box size=0.20569473673343697 0.603184882797648 0.6797492006351037
- link RightLeg: geometry collision box size=1.869166698216465 0.34190315219240996 0.12489818327934724; visual box size=1.869166698216465 0.34190315219240996 0.12489818327934724
- link RightLowerLeg: geometry collision box size=0.8343918814731542 0.46506786185183063 1.354342234914888; visual box size=0.8343918814731542 0.46506786185183063 1.354342234914888
Joints:
- joint Torso_BackLowerLeg: origin xyz=0 -2.1489674294037355 0 rpy=0 0 0 -> xyz=0 -1.7085554522910011 0 rpy=0 0 0
- joint Torso_FrontLowerLeg: origin xyz=0 2.1489674294037355 0 rpy=0 0 0 -> xyz=0 1.5157268514727786 0 rpy=0 0 0
- joint Torso_LeftLowerLeg: origin xyz=-2.646771162412283 0 0 rpy=0 0 0 -> xyz=-2.1483153574910983 0 0 rpy=0 0 0
- joint Torso_RightLowerLeg: origin xyz=2.646771162412283 0 0 rpy=0 0 0 -> xyz=1.869166698216465 0 0 rpy=0 0 0

File: body101.urdf (robot description, URDF)
Before this commit: robot robot, 9 links, 8 joints
Links:
- link BackLeg: geometry collision box size=0.1 2.0363057027227236 0.2000892112425181; visual box size=0.1 2.0363057027227236 0.2000892112425181
- link BackLowerLeg: geometry collision box size=0.39821387596722596 0.3092009707732883 0.9523641941971945; visual box size=0.39821387596722596 0.3092009707732883 0.9523641941971945
- link FrontLeg: geometry collision box size=0.28085824715357105 1.8503560791361886 0.27693777648130014; visual box size=0.28085824715357105 1.8503560791361886 0.27693777648130014
- link FrontLowerLeg: geometry collision box size=0.3217750955547207 0.11935172076918109 0.8798116869830762; visual box size=0.3217750955547207 0.11935172076918109 0.8798116869830762
- link LeftLeg: geometry collision box size=2.0740373341770657 0.1 0.1; visual box size=2.0740373341770657 0.1 0.1
- link LeftLowerLeg: geometry collision box size=0.1 0.1 1.1238030081344976; visual box size=0.1 0.1 1.1238030081344976
- link RightLeg: geometry collision box size=1.987219496873367 0.22649038790706624 0.13683906952417876; visual box size=1.987219496873367 0.22649038790706624 0.13683906952417876
- link RightLowerLeg: geometry collision box size=0.3078829276907665 0.15236926190898 1.0872961697707266; visual box size=0.3078829276907665 0.15236926190898 1.0872961697707266
Joints:
- joint Torso_BackLowerLeg: origin xyz=0 -1.8960074798007867 0 rpy=0 0 0 -> xyz=0 -2.0363057027227236 0 rpy=0 0 0
- joint Torso_FrontLowerLeg: origin xyz=0 1.8960074798007867 0 rpy=0 0 0 -> xyz=0 1.8503560791361886 0 rpy=0 0 0
- joint Torso_LeftLowerLeg: origin xyz=-2.0181264951686515 0 0 rpy=0 0 0 -> xyz=-2.0740373341770657 0 0 rpy=0 0 0
- joint Torso_RightLowerLeg: origin xyz=2.0181264951686515 0 0 rpy=0 0 0 -> xyz=1.987219496873367 0 0 rpy=0 0 0
