Commit message: For loop that goes through both symmetric and non symmetric and then graphs them both

File: body1010.urdf (robot description, URDF)
Before this commit: robot robot, 9 links, 8 joints
Links:
- link BackLeg: geometry collision box size=0.7854621885463178 1.9847869100097861 0.6907312929009901; visual box size=0.7854621885463178 1.9847869100097861 0.6907312929009901
- link BackLowerLeg: geometry collision box size=1.0277117567164917 0.19212907069857466 0.8106317751291774; visual box size=1.0277117567164917 0.19212907069857466 0.8106317751291774
- link FrontLeg: geometry collision box size=0.38570398348633433 1.9454736545702265 0.43125279632477564; visual box size=0.38570398348633433 1.9454736545702265 0.43125279632477564
- link FrontLowerLeg: geometry collision box size=0.1 0.35141433270871936 0.8684804144260372; visual box size=0.1 0.35141433270871936 0.8684804144260372
- link LeftLeg: geometry collision box size=2.751969294143779 0.4458662240179302 0.25030367841150525; visual box size=2.751969294143779 0.4458662240179302 0.25030367841150525
- link LeftLowerLeg: geometry collision box size=0.6264694671376403 0.21260687988998847 0.9565096229621071; visual box size=0.6264694671376403 0.21260687988998847 0.9565096229621071
- link RightLeg: geometry collision box size=1.4213085627655304 0.18222990657061267 0.1; visual box size=1.4213085627655304 0.18222990657061267 0.1
- link RightLowerLeg: geometry collision box size=0.45447837449601974 0.13823029574878334 1.0284186932690993; visual box size=0.45447837449601974 0.13823029574878334 1.0284186932690993
Joints:
- joint Torso_BackLowerLeg: origin xyz=0 -2.553750586626605 0 rpy=0 0 0 -> xyz=0 -1.9847869100097861 0 rpy=0 0 0
- joint Torso_FrontLowerLeg: origin xyz=0 2.553750586626605 0 rpy=0 0 0 -> xyz=0 1.9454736545702265 0 rpy=0 0 0
- joint Torso_LeftLowerLeg: origin xyz=-2.21822094143416 0 0 rpy=0 0 0 -> xyz=-2.751969294143779 0 0 rpy=0 0 0
- joint Torso_RightLowerLeg: origin xyz=2.21822094143416 0 0 rpy=0 0 0 -> xyz=1.4213085627655304 0 0 rpy=0 0 0

File: body1011.urdf (robot description, URDF)
Before this commit: robot robot, 9 links, 8 joints
Links:
- link BackLeg: geometry collision box size=0.37333313473348423 1.5898488168306821 0.14359252780906967; visual box size=0.37333313473348423 1.5898488168306821 0.14359252780906967
- link BackLowerLeg: geometry collision box size=0.2819149755211732 0.1 1.023781955750578; visual box size=0.2819149755211732 0.1 1.023781955750578
- link FrontLeg: geometry collision box size=0.1 2.2311224296546137 1.3285425692949189; visual box size=0.1 2.2311224296546137 1.3285425692949189
- link FrontLowerLeg: geometry collision box size=0.3953340160321137 0.20906377154324132 0.8348046210705248; visual box size=0.3953340160321137 0.20906377154324132 0.8348046210705248
- link LeftLeg: geometry collision box size=2.043672872155248 0.47785655576600694 0.553671690579892; visual box size=2.043672872155248 0.47785655576600694 0.553671690579892
- link LeftLowerLeg: geometry collision box size=0.4533258467488818 0.2089834891547869 0.560331372727411; visual box size=0.4533258467488818 0.2089834891547869 0.560331372727411
- link RightLeg: geometry collision box size=1.5262677126736575 0.47911140903751337 0.25825432153270855; visual box size=1.5262677126736575 0.47911140903751337 0.25825432153270855
- link RightLowerLeg: geometry collision box size=0.1 0.28494201635333644 1.5067707774332304; visual box size=0.1 0.28494201635333644 1.5067707774332304
Joints:
- joint Torso_BackLowerLeg: origin xyz=0 -2.2648833974189695 0 rpy=0 0 0 -> xyz=0 -1.5898488168306821 0 rpy=0 0 0
- joint Torso_FrontLowerLeg: origin xyz=0 2.2648833974189695 0 rpy=0 0 0 -> xyz=0 2.2311224296546137 0 rpy=0 0 0
- joint Torso_LeftLowerLeg: origin xyz=-2.234204869279888 0 0 rpy=0 0 0 -> xyz=-2.043672872155248 0 0 rpy=0 0 0
- joint Torso_RightLowerLeg: origin xyz=2.234204869279888 0 0 rpy=0 0 0 -> xyz=1.5262677126736575 0 0 rpy=0 0 0

File: body1012.urdf (robot description, URDF)
Before this commit: robot robot, 9 links, 8 joints
Links:
- link BackLeg: geometry collision box size=0.37163883423460264 1.872386169134143 0.21514923509549264; visual box size=0.37163883423460264 1.872386169134143 0.21514923509549264
- link BackLowerLeg: geometry collision box size=0.39717464641547034 0.1 1.0104826392459607; visual box size=0.39717464641547034 0.1 1.0104826392459607
- link FrontLeg: geometry collision box size=0.21172964137031203 1.8429139565103074 0.19654748610585285; visual box size=0.21172964137031203 1.8429139565103074 0.19654748610585285
- link FrontLowerLeg: geometry collision box size=0.2799928188939235 0.3606900570624958 0.9653821269638446; visual box size=0.2799928188939235 0.3606900570624958 0.9653821269638446
- link LeftLeg: geometry collision box size=2.1092361595804507 0.32101260506238855 0.1; visual box size=2.1092361595804507 0.32101260506238855 0.1
- link LeftLowerLeg: geometry collision box size=0.1 0.2986736989708883 1.0376298068155128; visual box size=0.1 0.2986736989708883 1.0376298068155128
- link RightLeg: geometry collision box size=2.116003155261186 0.1837145055526321 0.12450947997963767; visual box size=2.116003155261186 0.1837145055526321 0.12450947997963767
- link RightLowerLeg: geometry collision box size=0.1 0.20381989699645342 1.070052951353015; visual box size=0.1 0.20381989699645342 1.070052951353015
Joints:
- joint Torso_BackLowerLeg: origin xyz=0 -1.8825307201630852 0 rpy=0 0 0 -> xyz=0 -1.872386169134143 0 rpy=0 0 0
- joint Torso_FrontLowerLeg: origin xyz=0 1.8825307201630852 0 rpy=0 0 0 -> xyz=0 1.8429139565103074 0 rpy=0 0 0
- joint Torso_LeftLowerLeg: origin xyz=-2.1824890964487715 0 0 rpy=0 0 0 -> xyz=-2.1092361595804507 0 0 rpy=0 0 0
- joint Torso_RightLowerLeg: origin xyz=2.1824890964487715 0 0 rpy=0 0 0 -> xyz=2.116003155261186 0 0 rpy=0 0 0

File: body1013.urdf (robot description, URDF)
Before this commit: robot robot, 9 links, 8 joints
Links:
- link BackLeg: geometry collision box size=0.17350051627509877 1.945681190797078 0.3743946930927108; visual box size=0.17350051627509877 1.945681190797078 0.3743946930927108
- link BackLowerLeg: geometry collision box size=0.6042160002765141 0.1 1.1242739287403116; visual box size=0.6042160002765141 0.1 1.1242739287403116
- link FrontLeg: geometry collision box size=0.28869351333972637 2.198629070585942 0.1; visual box size=0.28869351333972637 2.198629070585942 0.1
- link FrontLowerLeg: geometry collision box size=0.5646203052651659 0.21151742132238738 0.8020924072479167; visual box size=0.5646203052651659 0.21151742132238738 0.8020924072479167
- link LeftLeg: geometry collision box size=2.0426211645418495 0.42907745529427543 0.3751874191886766; visual box size=2.0426211645418495 0.42907745529427543 0.3751874191886766
- link LeftLowerLeg: geometry collision box size=0.33530813215994315 0.6069385287249631 1.027016730906287; visual box size=0.33530813215994315 0.6069385287249631 1.027016730906287
- link RightLeg: geometry collision box size=2.2256847473527146 0.38801198774806445 0.347108559212823; visual box size=2.2256847473527146 0.38801198774806445 0.347108559212823
- link RightLowerLeg: geometry collision box size=0.1 0.1 1.0660284394575152; visual box size=0.1 0.1 1.0660284394575152
Joints:
- joint Torso_BackLowerLeg: origin xyz=0 -1.1763391472430456 0 rpy=0 0 0 -> xyz=0 -1.945681190797078 0 rpy=0 0 0
- joint Torso_FrontLowerLeg: origin xyz=0 1.1763391472430456 0 rpy=0 0 0 -> xyz=0 2.198629070585942 0 rpy=0 0 0
- joint Torso_LeftLowerLeg: origin xyz=-2.33536620899981 0 0 rpy=0 0 0 -> xyz=-2.0426211645418495 0 0 rpy=0 0 0
- joint Torso_RightLowerLeg: origin xyz=2.33536620899981 0 0 rpy=0 0 0 -> xyz=2.2256847473527146 0 0 rpy=0 0 0

File: body1014.urdf (robot description, URDF)
Before this commit: robot robot, 9 links, 8 joints
Links:
- link BackLeg: geometry collision box size=0.1 1.741855128514452 0.2453670106581766; visual box size=0.1 1.741855128514452 0.2453670106581766
- link BackLowerLeg: geometry collision box size=0.2637046844762737 0.1 1.7043918637938447; visual box size=0.2637046844762737 0.1 1.7043918637938447
- link FrontLeg: geometry collision box size=0.20936160123136838 1.5172530692915505 0.4142358698735193; visual box size=0.20936160123136838 1.5172530692915505 0.4142358698735193
- link FrontLowerLeg: geometry collision box size=0.610583550740484 0.24367891440445896 1.0746380343402568; visual box size=0.610583550740484 0.24367891440445896 1.0746380343402568
- link LeftLeg: geometry collision box size=2.256107459042827 0.21889470270402306 0.20541630034942257; visual box size=2.256107459042827 0.21889470270402306 0.20541630034942257
- link LeftLowerLeg: geometry collision box size=0.3041282347760436 0.17026756437201085 1.0106617664642987; visual box size=0.3041282347760436 0.17026756437201085 1.0106617664642987
- link RightLeg: geometry collision box size=1.9234387459263225 0.25813983117228734 0.4058539610897156; visual box size=1.9234387459263225 0.25813983117228734 0.4058539610897156
- link RightLowerLeg: geometry collision box size=0.6942803562030112 0.6860775533202375 1.1374148010861163; visual box size=0.6942803562030112 0.6860775533202375 1.1374148010861163
Joints:
- joint Torso_BackLowerLeg: origin xyz=0 -1.6703070180551407 0 rpy=0 0 0 -> xyz=0 -1.741855128514452 0 rpy=0 0 0
- joint Torso_FrontLowerLeg: origin xyz=0 1.6703070180551407 0 rpy=0 0 0 -> xyz=0 1.5172530692915505 0 rpy=0 0 0
- joint Torso_LeftLowerLeg: origin xyz=-2.76527945088786 0 0 rpy=0 0 0 -> xyz=-2.256107459042827 0 0 rpy=0 0 0
- joint Torso_RightLowerLeg: origin xyz=2.76527945088786 0 0 rpy=0 0 0 -> xyz=1.9234387459263225 0 0 rpy=0 0 0

File: body1015.urdf (robot description, URDF)
Before this commit: robot robot, 9 links, 8 joints
Links:
- link BackLeg: geometry collision box size=0.10948826300316297 1.9869253290766415 0.26031821527314813; visual box size=0.10948826300316297 1.9869253290766415 0.26031821527314813
- link BackLowerLeg: geometry collision box size=0.5188883792181329 0.1 1.1600944803400732; visual box size=0.5188883792181329 0.1 1.1600944803400732
- link FrontLeg: geometry collision box size=0.6278626740407511 1.9180996765891039 0.47985927513903964; visual box size=0.6278626740407511 1.9180996765891039 0.47985927513903964
- link FrontLowerLeg: geometry collision box size=0.5084342732747104 0.6543671160227158 0.8133003035151737; visual box size=0.5084342732747104 0.6543671160227158 0.8133003035151737
- link LeftLeg: geometry collision box size=1.4435365298265104 0.15909504921701725 0.5134427652921304; visual box size=1.4435365298265104 0.15909504921701725 0.5134427652921304
- link LeftLowerLeg: geometry collision box size=0.4919850685426438 0.1 0.9612576380816529; visual box size=0.4919850685426438 0.1 0.9612576380816529
- link RightLeg: geometry collision box size=1.8620304198000621 0.2327253951649326 0.1656530364447631; visual box size=1.8620304198000621 0.2327253951649326 0.1656530364447631
- link RightLowerLeg: geometry collision box size=0.36567200882625794 0.14975305470308592 1.1075387078588177; visual box size=0.36567200882625794 0.14975305470308592 1.1075387078588177
Joints:
- joint Torso_BackLowerLeg: origin xyz=0 -1.9606140448125386 0 rpy=0 0 0 -> xyz=0 -1.9869253290766415 0 rpy=0 0 0
- joint Torso_FrontLowerLeg: origin xyz=0 1.9606140448125386 0 rpy=0 0 0 -> xyz=0 1.9180996765891039 0 rpy=0 0 0
- joint Torso_LeftLowerLeg: origin xyz=-2.3374068674434154 0 0 rpy=0 0 0 -> xyz=-1.4435365298265104 0 0 rpy=0 0 0
- joint Torso_RightLowerLeg: origin xyz=2.3374068674434154 0 0 rpy=0 0 0 -> xyz=1.8620304198000621 0 0 rpy=0 0 0

File: body1016.urdf (robot description, URDF)
Before this commit: robot robot, 9 links, 8 joints
Links:
- link BackLeg: geometry collision box size=0.3165577370783994 2.2806230189362386 0.3641130401363573; visual box size=0.3165577370783994 2.2806230189362386 0.3641130401363573
- link BackLowerLeg: geometry collision box size=0.514813177470536 0.7975938752351122 1.7180941448953067; visual box size=0.514813177470536 0.7975938752351122 1.7180941448953067
- link FrontLeg: geometry collision box size=0.324879717175449 1.433150329505289 0.3263336653819391; visual box size=0.324879717175449 1.433150329505289 0.3263336653819391
- link FrontLowerLeg: geometry collision box size=0.2951573353134741 0.2569134074326787 1.5060194648954415; visual box size=0.2951573353134741 0.2569134074326787 1.5060194648954415
- link LeftLeg: geometry collision box size=2.222198648755183 0.1 0.8337468686328162; visual box size=2.222198648755183 0.1 0.8337468686328162
- link LeftLowerLeg: geometry collision box size=0.1 0.10394557413035738 1.3702650780994368; visual box size=0.1 0.10394557413035738 1.3702650780994368
- link RightLeg: geometry collision box size=1.133324078812467 0.65793761156519 0.323409626103307; visual box size=1.133324078812467 0.65793761156519 0.323409626103307
- link RightLowerLeg: geometry collision box size=0.6171224076354429 0.672718627095976 1.8368171275391227; visual box size=0.6171224076354429 0.672718627095976 1.8368171275391227
Joints:
- joint Torso_BackLowerLeg: origin xyz=0 -2.590380794455892 0 rpy=0 0 0 -> xyz=0 -2.2806230189362386 0 rpy=0 0 0
- joint Torso_FrontLowerLeg: origin xyz=0 2.590380794455892 0 rpy=0 0 0 -> xyz=0 1.433150329505289 0 rpy=0 0 0
- joint Torso_LeftLowerLeg: origin xyz=-2.177424438008144 0 0 rpy=0 0 0 -> xyz=-2.222198648755183 0 0 rpy=0 0 0
- joint Torso_RightLowerLeg: origin xyz=2.177424438008144 0 0 rpy=0 0 0 -> xyz=1.133324078812467 0 0 rpy=0 0 0

File: body1017.urdf (robot description, URDF)
Before this commit: robot robot, 9 links, 8 joints
Links:
- link BackLeg: geometry collision box size=0.41730376012140924 0.9252439634236385 0.22740582285208852; visual box size=0.41730376012140924 0.9252439634236385 0.22740582285208852
- link BackLowerLeg: geometry collision box size=0.1263717289553047 0.21293341249670927 0.6447754309207602; visual box size=0.1263717289553047 0.21293341249670927 0.6447754309207602
- link FrontLeg: geometry collision box size=0.27812011116828733 2.1373287382847863 0.49552997210428956; visual box size=0.27812011116828733 2.1373287382847863 0.49552997210428956
- link FrontLowerLeg: geometry collision box size=0.1 0.18201315039479324 1.2714511172694627; visual box size=0.1 0.18201315039479324 1.2714511172694627
- link LeftLeg: geometry collision box size=2.1166154933835144 0.29562096762682977 0.1; visual box size=2.1166154933835144 0.29562096762682977 0.1
- link LeftLowerLeg: geometry collision box size=0.17496171043896244 0.1 1.0007429235823304; visual box size=0.17496171043896244 0.1 1.0007429235823304
- link RightLeg: geometry collision box size=1.939559843201718 0.2751452843252913 0.42886073692905835; visual box size=1.939559843201718 0.2751452843252913 0.42886073692905835
- link RightLowerLeg: geometry collision box size=1.2298128463702858 1.110668199346398 1.6710581651118241; visual box size=1.2298128463702858 1.110668199346398 1.6710581651118241
Joints:
- joint Torso_BackLowerLeg: origin xyz=0 -2.0227582421268138 0 rpy=0 0 0 -> xyz=0 -0.9252439634236385 0 rpy=0 0 0
- joint Torso_FrontLowerLeg: origin xyz=0 2.0227582421268138 0 rpy=0 0 0 -> xyz=0 2.1373287382847863 0 rpy=0 0 0
- joint Torso_LeftLowerLeg: origin xyz=-2.1714043496212163 0 0 rpy=0 0 0 -> xyz=-2.1166154933835144 0 0 rpy=0 0 0
- joint Torso_RightLowerLeg: origin xyz=2.1714043496212163 0 0 rpy=0 0 0 -> xyz=1.939559843201718 0 0 rpy=0 0 0
