Commit message: milestone3

File: body1.urdf (robot description, URDF)
Before this commit: robot robot, 9 links, 8 joints
Links:
- link FrontLowerLeg: geometry collision box size=0.2 0.2 1; visual box size=0.2 0.2 1
- link LeftLowerLeg: geometry collision box size=0.2 0.2 1; visual box size=0.2 0.2 1
- link RightLowerLeg: geometry collision box size=0.2 0.2 1; visual box size=0.2 0.2 1

File: body5.urdf (robot description, URDF)
Before this commit: robot robot, 9 links, 8 joints
Links:
- link BackLeg: geometry collision box size=0.2 2 0.2; visual box size=0.2 2 0.2
- link BackLowerLeg: geometry collision box size=0.2 0.2 1; visual box size=0.2 0.2 1
- link FrontLeg: geometry collision box size=0.2 2 0.2; visual box size=0.2 2 0.2
- link FrontLowerLeg: geometry collision box size=0.2 0.2 1; visual box size=0.2 0.2 1
- link LeftLeg: geometry collision box size=2 0.2 0.2; visual box size=2 0.2 0.2
- link LeftLowerLeg: geometry collision box size=0.2 0.2 1; visual box size=0.2 0.2 1
- link RightLeg: geometry collision box size=2 0.2 0.2; visual box size=2 0.2 0.2
- link RightLowerLeg: geometry collision box size=0.2 0.2 1; visual box size=0.2 0.2 1
Joints:
- joint Torso_BackLowerLeg: origin xyz=0 -1.9746695689187843 0 rpy=0 0 0 -> xyz=0 -2 0 rpy=0 0 0
- joint Torso_FrontLowerLeg: origin xyz=0 2.0 0 rpy=0 0 0 -> xyz=0 2 0 rpy=0 0 0
- joint Torso_LeftLowerLeg: origin xyz=-1.990996342904461 0 0 rpy=0 0 0 -> xyz=-2 0 0 rpy=0 0 0
- joint Torso_RightLowerLeg: origin xyz=2.0 0 0 rpy=0 0 0 -> xyz=2 0 0 rpy=0 0 0

File: body6.urdf (robot description, URDF)
Before this commit: robot robot, 9 links, 8 joints
Links:
- link BackLeg: geometry collision box size=0.2 2 0.2; visual box size=0.2 2 0.2
- link BackLowerLeg: geometry collision box size=0.2 0.2 1; visual box size=0.2 0.2 1
- link FrontLeg: geometry collision box size=0.2 2 0.2; visual box size=0.2 2 0.2
- link FrontLowerLeg: geometry collision box size=0.2 0.2 1; visual box size=0.2 0.2 1
- link LeftLeg: geometry collision box size=2 0.2 0.2; visual box size=2 0.2 0.2
- link LeftLowerLeg: geometry collision box size=0.2 0.2 1; visual box size=0.2 0.2 1
- link RightLeg: geometry collision box size=2 0.2 0.2; visual box size=2 0.2 0.2
- link RightLowerLeg: geometry collision box size=0.2 0.2 1; visual box size=0.2 0.2 1
Joints:
- joint Torso_BackLowerLeg: origin xyz=0 -2.0 0 rpy=0 0 0 -> xyz=0 -2 0 rpy=0 0 0
- joint Torso_FrontLowerLeg: origin xyz=0 1.8448889396967072 0 rpy=0 0 0 -> xyz=0 2 0 rpy=0 0 0
- joint Torso_LeftLowerLeg: origin xyz=-1.8684050711148505 0 0 rpy=0 0 0 -> xyz=-2 0 0 rpy=0 0 0
- joint Torso_RightLowerLeg: origin xyz=2.0 0 0 rpy=0 0 0 -> xyz=2 0 0 rpy=0 0 0

File: body7.urdf (robot description, URDF)
Before this commit: robot robot, 9 links, 8 joints
Links:
- link BackLeg: geometry collision box size=0.2 2 0.2; visual box size=0.2 2 0.2
- link BackLowerLeg: geometry collision box size=0.2 0.2 1; visual box size=0.2 0.2 1
- link FrontLeg: geometry collision box size=0.2 2 0.2; visual box size=0.2 2 0.2
- link FrontLowerLeg: geometry collision box size=0.2 0.2 1; visual box size=0.2 0.2 1
- link LeftLeg: geometry collision box size=2 0.2 0.2; visual box size=2 0.2 0.2
- link LeftLowerLeg: geometry collision box size=0.2 0.2 1; visual box size=0.2 0.2 1
- link RightLeg: geometry collision box size=2 0.2 0.2; visual box size=2 0.2 0.2
- link RightLowerLeg: geometry collision box size=0.2 0.2 1; visual box size=0.2 0.2 1
Joints:
- joint Torso_BackLowerLeg: origin xyz=0 -2.0 0 rpy=0 0 0 -> xyz=0 -2 0 rpy=0 0 0
- joint Torso_FrontLowerLeg: origin xyz=0 2.0 0 rpy=0 0 0 -> xyz=0 2 0 rpy=0 0 0
- joint Torso_LeftLowerLeg: origin xyz=-1.9147555050317053 0 0 rpy=0 0 0 -> xyz=-2 0 0 rpy=0 0 0
- joint Torso_RightLowerLeg: origin xyz=2.0 0 0 rpy=0 0 0 -> xyz=2 0 0 rpy=0 0 0

File: body8.urdf (robot description, URDF)
Before this commit: robot robot, 9 links, 8 joints
Links:
- link BackLeg: geometry collision box size=0.2 2 0.2; visual box size=0.2 2 0.2
- link BackLowerLeg: geometry collision box size=0.2 0.2 1; visual box size=0.2 0.2 1
- link FrontLeg: geometry collision box size=0.2 2 0.2; visual box size=0.2 2 0.2
- link FrontLowerLeg: geometry collision box size=0.2 0.2 1; visual box size=0.2 0.2 1
- link LeftLeg: geometry collision box size=2 0.2 0.2; visual box size=2 0.2 0.2
- link LeftLowerLeg: geometry collision box size=0.2 0.2 1; visual box size=0.2 0.2 1
- link RightLeg: geometry collision box size=2 0.2 0.2; visual box size=2 0.2 0.2
- link RightLowerLeg: geometry collision box size=0.2 0.2 1; visual box size=0.2 0.2 1
Joints:
- joint Torso_BackLowerLeg: origin xyz=0 -2.0 0 rpy=0 0 0 -> xyz=0 -2 0 rpy=0 0 0
- joint Torso_FrontLowerLeg: origin xyz=0 2.0 0 rpy=0 0 0 -> xyz=0 2 0 rpy=0 0 0
- joint Torso_LeftLowerLeg: origin xyz=-2.0 0 0 rpy=0 0 0 -> xyz=-2 0 0 rpy=0 0 0
- joint Torso_RightLowerLeg: origin xyz=2.0 0 0 rpy=0 0 0 -> xyz=2 0 0 rpy=0 0 0

File: body9.urdf (robot description, URDF)
Before this commit: robot robot, 9 links, 8 joints
Links:
- link BackLeg: geometry collision box size=0.2 2 0.2; visual box size=0.2 2 0.2
- link BackLowerLeg: geometry collision box size=0.2 0.2 1; visual box size=0.2 0.2 1
- link FrontLeg: geometry collision box size=0.2 2 0.2; visual box size=0.2 2 0.2
- link FrontLowerLeg: geometry collision box size=0.2 0.2 1; visual box size=0.2 0.2 1
- link LeftLeg: geometry collision box size=2 0.2 0.2; visual box size=2 0.2 0.2
- link LeftLowerLeg: geometry collision box size=0.2 0.2 1; visual box size=0.2 0.2 1
- link RightLeg: geometry collision box size=2 0.2 0.2; visual box size=2 0.2 0.2
- link RightLowerLeg: geometry collision box size=0.2 0.2 1; visual box size=0.2 0.2 1
Joints:
- joint Torso_BackLowerLeg: origin xyz=0 -2.0 0 rpy=0 0 0 -> xyz=0 -2 0 rpy=0 0 0
- joint Torso_FrontLowerLeg: origin xyz=0 2.0 0 rpy=0 0 0 -> xyz=0 2 0 rpy=0 0 0
- joint Torso_LeftLowerLeg: origin xyz=-1.9029732146247642 0 0 rpy=0 0 0 -> xyz=-2 0 0 rpy=0 0 0
- joint Torso_RightLowerLeg: origin xyz=1.8720823936861066 0 0 rpy=0 0 0 -> xyz=2 0 0 rpy=0 0 0
