Commit message: done

File: body1.urdf (robot description, URDF)
Before this commit: robot robot, 9 links, 8 joints
Links:
- link BackLeg: geometry collision box size=0.29321627871047296 1.634216622388374 0.1808519939751103; visual box size=0.29321627871047296 1.634216622388374 0.1808519939751103
- link BackLowerLeg: geometry collision box size=0.7891181142260446 0.6923323519804043 2.431855426523922; visual box size=0.7891181142260446 0.6923323519804043 2.431855426523922
- link FrontLeg: geometry collision box size=0.9409332437018874 1.0182488757272599 0.1476871819205267; visual box size=0.9409332437018874 1.0182488757272599 0.1476871819205267
- link FrontLowerLeg: geometry collision box size=0.20043704672069843 0.6556649121699412 2.6227232657514015; visual box size=0.20043704672069843 0.6556649121699412 2.6227232657514015
- link LeftLeg: geometry collision box size=2.755863730401788 0.33019087734455116 0.28155249316981545; visual box size=2.755863730401788 0.33019087734455116 0.28155249316981545
- link LeftLowerLeg: geometry collision box size=0.1 0.5689296780757456 0.13061609261170445; visual box size=0.1 0.5689296780757456 0.13061609261170445
- link RightLeg: geometry collision box size=1.666052938186125 0.1 0.28693755146402666; visual box size=1.666052938186125 0.1 0.28693755146402666
- link RightLowerLeg: geometry collision box size=0.789460428861575 0.2623468341620847 2.4930029917886887; visual box size=0.789460428861575 0.2623468341620847 2.4930029917886887
Joints:
- joint Torso_BackLowerLeg: origin xyz=0 -2 0 rpy=0 0 0 -> xyz=0 -1.634216622388374 0 rpy=0 0 0
- joint Torso_FrontLowerLeg: origin xyz=0 2 0 rpy=0 0 0 -> xyz=0 1.0182488757272599 0 rpy=0 0 0
- joint Torso_LeftLowerLeg: origin xyz=-2 0 0 rpy=0 0 0 -> xyz=-2.755863730401788 0 0 rpy=0 0 0
- joint Torso_RightLowerLeg: origin xyz=2 0 0 rpy=0 0 0 -> xyz=1.666052938186125 0 0 rpy=0 0 0

File: body100.urdf (robot description, URDF)
Before this commit: robot robot, 9 links, 8 joints
Links:
- link BackLeg: geometry collision box size=0.1 1.8027373542778888 0.13794610198998994; visual box size=0.1 1.8027373542778888 0.13794610198998994
- link BackLowerLeg: geometry collision box size=0.7400040365470731 0.8536770163881522 2.318699544319395; visual box size=0.7400040365470731 0.8536770163881522 2.318699544319395
- link FrontLeg: geometry collision box size=0.975244365777288 0.9887597183723452 0.29002574043998114; visual box size=0.975244365777288 0.9887597183723452 0.29002574043998114
- link FrontLowerLeg: geometry collision box size=0.1601642894859361 0.48145959584809195 2.5018471600212684; visual box size=0.1601642894859361 0.48145959584809195 2.5018471600212684
- link LeftLeg: geometry collision box size=2.8368744674031303 0.4869492425814484 0.21548768012634212; visual box size=2.8368744674031303 0.4869492425814484 0.21548768012634212
- link LeftLowerLeg: geometry collision box size=0.1 0.6443284274712835 0.1; visual box size=0.1 0.6443284274712835 0.1
- link RightLeg: geometry collision box size=1.5172089507079338 0.1 0.43246111643986845; visual box size=1.5172089507079338 0.1 0.43246111643986845
- link RightLowerLeg: geometry collision box size=0.9495897123289279 0.40650688478997443 2.686674666695743; visual box size=0.9495897123289279 0.40650688478997443 2.686674666695743
Joints:
- joint Torso_BackLowerLeg: origin xyz=0 -2.0116093912968154 0 rpy=0 0 0 -> xyz=0 -1.8027373542778888 0 rpy=0 0 0
- joint Torso_FrontLowerLeg: origin xyz=0 2.1117779375669974 0 rpy=0 0 0 -> xyz=0 0.9887597183723452 0 rpy=0 0 0
- joint Torso_LeftLowerLeg: origin xyz=-1.8798969393669138 0 0 rpy=0 0 0 -> xyz=-2.8368744674031303 0 0 rpy=0 0 0
- joint Torso_RightLowerLeg: origin xyz=1.949407073601662 0 0 rpy=0 0 0 -> xyz=1.5172089507079338 0 0 rpy=0 0 0

File: body101.urdf (robot description, URDF)
Before this commit: robot robot, 9 links, 8 joints
Links:
- link BackLeg: geometry collision box size=0.23047229295693492 1.6245099035301795 0.29567739264607484; visual box size=0.23047229295693492 1.6245099035301795 0.29567739264607484
- link BackLowerLeg: geometry collision box size=0.9171635496532544 0.7699594616679548 2.5419796460413; visual box size=0.9171635496532544 0.7699594616679548 2.5419796460413
- link FrontLeg: geometry collision box size=1.0428627520648925 0.9617672896349357 0.2867250283349388; visual box size=1.0428627520648925 0.9617672896349357 0.2867250283349388
- link FrontLowerLeg: geometry collision box size=0.20090577217876737 0.537059075589671 2.4807478726292174; visual box size=0.20090577217876737 0.537059075589671 2.4807478726292174
- link LeftLeg: geometry collision box size=2.7494804276562297 0.139060251882468 0.22916416908800094; visual box size=2.7494804276562297 0.139060251882468 0.22916416908800094
- link LeftLowerLeg: geometry collision box size=0.2820058970050292 0.7102436797810432 0.1; visual box size=0.2820058970050292 0.7102436797810432 0.1
- link RightLeg: geometry collision box size=1.5388810819324452 0.21030823582881555 0.18730606699172342; visual box size=1.5388810819324452 0.21030823582881555 0.18730606699172342
- link RightLowerLeg: geometry collision box size=0.9814264801866495 0.41323939605662957 2.296671949513536; visual box size=0.9814264801866495 0.41323939605662957 2.296671949513536
Joints:
- joint Torso_BackLowerLeg: origin xyz=0 -2.0363057027227236 0 rpy=0 0 0 -> xyz=0 -1.6245099035301795 0 rpy=0 0 0
- joint Torso_FrontLowerLeg: origin xyz=0 1.8503560791361886 0 rpy=0 0 0 -> xyz=0 0.9617672896349357 0 rpy=0 0 0
- joint Torso_LeftLowerLeg: origin xyz=-2.0740373341770657 0 0 rpy=0 0 0 -> xyz=-2.7494804276562297 0 0 rpy=0 0 0
- joint Torso_RightLowerLeg: origin xyz=1.987219496873367 0 0 rpy=0 0 0 -> xyz=1.5388810819324452 0 0 rpy=0 0 0

File: body102.urdf (robot description, URDF)
Before this commit: robot robot, 9 links, 8 joints
Links:
- link BackLeg: geometry collision box size=0.34752608143284053 1.7965683882135917 0.1; visual box size=0.34752608143284053 1.7965683882135917 0.1
- link BackLowerLeg: geometry collision box size=0.8029537730928717 0.6075746419242427 2.4395309817545026; visual box size=0.8029537730928717 0.6075746419242427 2.4395309817545026
- link FrontLeg: geometry collision box size=1.0900439077017614 0.834756603184776 0.1; visual box size=1.0900439077017614 0.834756603184776 0.1
- link FrontLowerLeg: geometry collision box size=0.17925327987280462 0.8022501965154465 2.5376564493560085; visual box size=0.17925327987280462 0.8022501965154465 2.5376564493560085
- link LeftLeg: geometry collision box size=2.90996895138055 0.5227922128414367 0.31819839503052433; visual box size=2.90996895138055 0.5227922128414367 0.31819839503052433
- link LeftLowerLeg: geometry collision box size=0.14619903510759819 0.7455805801866372 0.14140180902148555; visual box size=0.14619903510759819 0.7455805801866372 0.14140180902148555
- link RightLeg: geometry collision box size=1.8022617903043867 0.12244977360238182 0.35480197069433234; visual box size=1.8022617903043867 0.12244977360238182 0.35480197069433234
- link RightLowerLeg: geometry collision box size=0.7039612374542517 0.1 2.2976648142606915; visual box size=0.7039612374542517 0.1 2.2976648142606915
Joints:
- joint Torso_BackLowerLeg: origin xyz=0 -1.8298718576544903 0 rpy=0 0 0 -> xyz=0 -1.7965683882135917 0 rpy=0 0 0
- joint Torso_FrontLowerLeg: origin xyz=0 2.0472667344106386 0 rpy=0 0 0 -> xyz=0 0.834756603184776 0 rpy=0 0 0
- joint Torso_LeftLowerLeg: origin xyz=-2.23519797648998 0 0 rpy=0 0 0 -> xyz=-2.90996895138055 0 0 rpy=0 0 0
- joint Torso_RightLowerLeg: origin xyz=2.046071392741286 0 0 rpy=0 0 0 -> xyz=1.8022617903043867 0 0 rpy=0 0 0

File: body103.urdf (robot description, URDF)
Before this commit: robot robot, 9 links, 8 joints
Links:
- link BackLeg: geometry collision box size=0.23357396254266075 1.6713314904018473 0.20337429099169915; visual box size=0.23357396254266075 1.6713314904018473 0.20337429099169915
- link BackLowerLeg: geometry collision box size=0.9166889514917627 0.5587912687751547 2.4216164517320724; visual box size=0.9166889514917627 0.5587912687751547 2.4216164517320724
- link FrontLeg: geometry collision box size=0.7527388503225662 0.8855779958053309 0.1; visual box size=0.7527388503225662 0.8855779958053309 0.1
- link FrontLowerLeg: geometry collision box size=0.1323808070700598 0.5239970671429098 2.6797665402958284; visual box size=0.1323808070700598 0.5239970671429098 2.6797665402958284
- link LeftLeg: geometry collision box size=2.646544524439188 0.1692047928539095 0.1; visual box size=2.646544524439188 0.1692047928539095 0.1
- link LeftLowerLeg: geometry collision box size=0.1 0.46576755342331244 0.18967918764918648; visual box size=0.1 0.46576755342331244 0.18967918764918648
- link RightLeg: geometry collision box size=1.52791677432567 0.1 0.46739570358177107; visual box size=1.52791677432567 0.1 0.46739570358177107
- link RightLowerLeg: geometry collision box size=0.8361543380900951 0.32605385063962056 2.6247965297661033; visual box size=0.8361543380900951 0.32605385063962056 2.6247965297661033
Joints:
- joint Torso_BackLowerLeg: origin xyz=0 -2.1047713212329273 0 rpy=0 0 0 -> xyz=0 -1.6713314904018473 0 rpy=0 0 0
- joint Torso_FrontLowerLeg: origin xyz=0 2.190597673679498 0 rpy=0 0 0 -> xyz=0 0.8855779958053309 0 rpy=0 0 0
- joint Torso_LeftLowerLeg: origin xyz=-1.9680173841222657 0 0 rpy=0 0 0 -> xyz=-2.646544524439188 0 0 rpy=0 0 0
- joint Torso_RightLowerLeg: origin xyz=1.8877914978419268 0 0 rpy=0 0 0 -> xyz=1.52791677432567 0 0 rpy=0 0 0

File: body104.urdf (robot description, URDF)
Before this commit: robot robot, 9 links, 8 joints
Links:
- link BackLeg: geometry collision box size=0.2089921407125166 1.6994633284127132 0.20032192025346862; visual box size=0.2089921407125166 1.6994633284127132 0.20032192025346862
- link BackLowerLeg: geometry collision box size=0.9200757886219646 0.5786512212907359 2.3615152786928277; visual box size=0.9200757886219646 0.5786512212907359 2.3615152786928277
- link FrontLeg: geometry collision box size=0.7837576746615734 1.1852413898705598 0.1; visual box size=0.7837576746615734 1.1852413898705598 0.1
- link FrontLowerLeg: geometry collision box size=0.12257598860446876 0.7258529087909091 2.5557826160162573; visual box size=0.12257598860446876 0.7258529087909091 2.5557826160162573
- link LeftLeg: geometry collision box size=2.830723632679263 0.1892699908532018 0.41343259510054525; visual box size=2.830723632679263 0.1892699908532018 0.41343259510054525
- link LeftLowerLeg: geometry collision box size=0.1 0.554270912978266 0.13616678430338033; visual box size=0.1 0.554270912978266 0.13616678430338033
- link RightLeg: geometry collision box size=1.6615178637577874 0.1 0.2737375106914265; visual box size=1.6615178637577874 0.1 0.2737375106914265
- link RightLowerLeg: geometry collision box size=0.6527910665336848 0.1 2.607592049141297; visual box size=0.6527910665336848 0.1 2.607592049141297
Joints:
- joint Torso_BackLowerLeg: origin xyz=0 -1.846555874854684 0 rpy=0 0 0 -> xyz=0 -1.6994633284127132 0 rpy=0 0 0
- joint Torso_FrontLowerLeg: origin xyz=0 2.151675507139278 0 rpy=0 0 0 -> xyz=0 1.1852413898705598 0 rpy=0 0 0
- joint Torso_LeftLowerLeg: origin xyz=-1.9742868777177178 0 0 rpy=0 0 0 -> xyz=-2.830723632679263 0 0 rpy=0 0 0
- joint Torso_RightLowerLeg: origin xyz=2.0784403870776544 0 0 rpy=0 0 0 -> xyz=1.6615178637577874 0 0 rpy=0 0 0

File: body105.urdf (robot description, URDF)
Before this commit: robot robot, 9 links, 8 joints
Links:
- link BackLeg: geometry collision box size=0.3389189163695856 1.4969490301552786 0.12936200930659225; visual box size=0.3389189163695856 1.4969490301552786 0.12936200930659225
- link BackLowerLeg: geometry collision box size=0.6573312783005002 0.5873411360254657 2.4868134582553103; visual box size=0.6573312783005002 0.5873411360254657 2.4868134582553103
- link FrontLeg: geometry collision box size=0.7751522790781351 0.9270876529973073 0.2671906275422936; visual box size=0.7751522790781351 0.9270876529973073 0.2671906275422936
- link FrontLowerLeg: geometry collision box size=0.2500633229480518 0.7420011152234708 2.7276528973943646; visual box size=0.2500633229480518 0.7420011152234708 2.7276528973943646
- link LeftLeg: geometry collision box size=2.8165856584639246 0.32225830054360344 0.1; visual box size=2.8165856584639246 0.32225830054360344 0.1
- link LeftLowerLeg: geometry collision box size=0.1820806320267878 0.6666873749833861 0.1; visual box size=0.1820806320267878 0.6666873749833861 0.1
- link RightLeg: geometry collision box size=1.6181526266004165 0.10086930434285826 0.3558635190449309; visual box size=1.6181526266004165 0.10086930434285826 0.3558635190449309
- link RightLowerLeg: geometry collision box size=0.9582497929326974 0.20310434769210284 2.5725090084741797; visual box size=0.9582497929326974 0.20310434769210284 2.5725090084741797
Joints:
- joint Torso_BackLowerLeg: origin xyz=0 -1.7737380945319077 0 rpy=0 0 0 -> xyz=0 -1.4969490301552786 0 rpy=0 0 0
- joint Torso_FrontLowerLeg: origin xyz=0 2.135679644365217 0 rpy=0 0 0 -> xyz=0 0.9270876529973073 0 rpy=0 0 0
- joint Torso_LeftLowerLeg: origin xyz=-2.329654183237884 0 0 rpy=0 0 0 -> xyz=-2.8165856584639246 0 0 rpy=0 0 0
- joint Torso_RightLowerLeg: origin xyz=1.7905444023457677 0 0 rpy=0 0 0 -> xyz=1.6181526266004165 0 0 rpy=0 0 0

File: body106.urdf (robot description, URDF)
Before this commit: robot robot, 9 links, 8 joints
Links:
- link BackLeg: geometry collision box size=0.4848307667342037 1.695099802172592 0.11473836025631284; visual box size=0.4848307667342037 1.695099802172592 0.11473836025631284
- link BackLowerLeg: geometry collision box size=0.6745779265268628 0.7738776582816018 2.4836799019680074; visual box size=0.6745779265268628 0.7738776582816018 2.4836799019680074
- link FrontLeg: geometry collision box size=0.8328427108422848 1.075253120831047 0.2805053609296874; visual box size=0.8328427108422848 1.075253120831047 0.2805053609296874
- link FrontLowerLeg: geometry collision box size=0.16743908263154803 0.58434188650283 2.6350798822638204; visual box size=0.16743908263154803 0.58434188650283 2.6350798822638204
- link LeftLeg: geometry collision box size=2.858564121893701 0.2612982043451809 0.14008637002993804; visual box size=2.858564121893701 0.2612982043451809 0.14008637002993804
- link LeftLowerLeg: geometry collision box size=0.15423547788105477 0.45880102440642473 0.2519058945146978; visual box size=0.15423547788105477 0.45880102440642473 0.2519058945146978
- link RightLeg: geometry collision box size=1.57557655775494 0.1 0.27245277750904673; visual box size=1.57557655775494 0.1 0.27245277750904673
- link RightLowerLeg: geometry collision box size=0.9181795271002839 0.4301750355563439 2.37350057788013; visual box size=0.9181795271002839 0.4301750355563439 2.37350057788013
Joints:
- joint Torso_BackLowerLeg: origin xyz=0 -2.440544926884705 0 rpy=0 0 0 -> xyz=0 -1.695099802172592 0 rpy=0 0 0
- joint Torso_FrontLowerLeg: origin xyz=0 1.9146577663332196 0 rpy=0 0 0 -> xyz=0 1.075253120831047 0 rpy=0 0 0
- joint Torso_LeftLowerLeg: origin xyz=-2.362644132696421 0 0 rpy=0 0 0 -> xyz=-2.858564121893701 0 0 rpy=0 0 0
- joint Torso_RightLowerLeg: origin xyz=2.0036338645258005 0 0 rpy=0 0 0 -> xyz=1.57557655775494 0 0 rpy=0 0 0

File: body107.urdf (robot description, URDF)
Before this commit: robot robot, 9 links, 8 joints
Links:
- link BackLeg: geometry collision box size=0.11115738841970357 1.6926068414790403 0.1; visual box size=0.11115738841970357 1.6926068414790403 0.1
- link BackLowerLeg: geometry collision box size=0.6306612996609052 0.8477367286666095 2.262226637314429; visual box size=0.6306612996609052 0.8477367286666095 2.262226637314429
- link FrontLeg: geometry collision box size=0.8269774809262888 1.0449153605048047 0.1; visual box size=0.8269774809262888 1.0449153605048047 0.1
- link FrontLowerLeg: geometry collision box size=0.3656609493254813 0.6370212074606869 2.430353883910703; visual box size=0.3656609493254813 0.6370212074606869 2.430353883910703
- link LeftLeg: geometry collision box size=2.8598262337802702 0.22495507682330057 0.1730980958857663; visual box size=2.8598262337802702 0.22495507682330057 0.1730980958857663
- link LeftLowerLeg: geometry collision box size=0.19704983059386974 0.42271103499415175 0.1; visual box size=0.19704983059386974 0.42271103499415175 0.1
- link RightLeg: geometry collision box size=1.6606537575448814 0.1 0.18198948958019867; visual box size=1.6606537575448814 0.1 0.18198948958019867
- link RightLowerLeg: geometry collision box size=0.7282869501123039 0.257884233851781 2.578551478339681; visual box size=0.7282869501123039 0.257884233851781 2.578551478339681
Joints:
- joint Torso_BackLowerLeg: origin xyz=0 -1.9567455392121007 0 rpy=0 0 0 -> xyz=0 -1.6926068414790403 0 rpy=0 0 0
- joint Torso_FrontLowerLeg: origin xyz=0 2.041619855289006 0 rpy=0 0 0 -> xyz=0 1.0449153605048047 0 rpy=0 0 0
- joint Torso_LeftLowerLeg: origin xyz=-1.8825068386492514 0 0 rpy=0 0 0 -> xyz=-2.8598262337802702 0 0 rpy=0 0 0
- joint Torso_RightLowerLeg: origin xyz=1.989649961158117 0 0 rpy=0 0 0 -> xyz=1.6606537575448814 0 0 rpy=0 0 0

File: body108.urdf (robot description, URDF)
Before this commit: robot robot, 9 links, 8 joints
Links:
- link BackLeg: geometry collision box size=0.2069649514722015 1.4631965307920574 0.14314283227539437; visual box size=0.2069649514722015 1.4631965307920574 0.14314283227539437
- link BackLowerLeg: geometry collision box size=0.7011974729998488 0.7089761068089754 2.438771793163391; visual box size=0.7011974729998488 0.7089761068089754 2.438771793163391
- link FrontLeg: geometry collision box size=0.7430493703551394 0.8418695771824383 0.2958390780592533; visual box size=0.7430493703551394 0.8418695771824383 0.2958390780592533
- link FrontLowerLeg: geometry collision box size=0.1 0.8529453830238569 2.509217549476979; visual box size=0.1 0.8529453830238569 2.509217549476979
- link LeftLeg: geometry collision box size=2.7272657245059126 0.38200026829903316 0.2155878694444049; visual box size=2.7272657245059126 0.38200026829903316 0.2155878694444049
- link LeftLowerLeg: geometry collision box size=0.1 0.681586553474371 0.1; visual box size=0.1 0.681586553474371 0.1
- link RightLeg: geometry collision box size=1.6766627531540408 0.2840586970507525 0.2942285936246058; visual box size=1.6766627531540408 0.2840586970507525 0.2942285936246058
- link RightLowerLeg: geometry collision box size=0.8896289952868278 0.32212920515550836 2.376939512959673; visual box size=0.8896289952868278 0.32212920515550836 2.376939512959673
Joints:
- joint Torso_BackLowerLeg: origin xyz=0 -2.189904112134409 0 rpy=0 0 0 -> xyz=0 -1.4631965307920574 0 rpy=0 0 0
- joint Torso_FrontLowerLeg: origin xyz=0 2.104779401995508 0 rpy=0 0 0 -> xyz=0 0.8418695771824383 0 rpy=0 0 0
- joint Torso_LeftLowerLeg: origin xyz=-2.0344949779641803 0 0 rpy=0 0 0 -> xyz=-2.7272657245059126 0 0 rpy=0 0 0
- joint Torso_RightLowerLeg: origin xyz=2.0837749321172834 0 0 rpy=0 0 0 -> xyz=1.6766627531540408 0 0 rpy=0 0 0

File: body109.urdf (robot description, URDF)
Before this commit: robot robot, 9 links, 8 joints
Links:
- link BackLeg: geometry collision box size=0.10539221347866229 1.58913512194184 0.348341746819507; visual box size=0.10539221347866229 1.58913512194184 0.348341746819507
- link BackLowerLeg: geometry collision box size=0.872675476960604 0.5131492372603348 2.2960688066497292; visual box size=0.872675476960604 0.5131492372603348 2.2960688066497292
- link FrontLeg: geometry collision box size=0.8738777328698409 1.0182689891632226 0.25915458302561334; visual box size=0.8738777328698409 1.0182689891632226 0.25915458302561334
- link FrontLowerLeg: geometry collision box size=0.19648442089349655 0.6870131543627426 2.7759090872853025; visual box size=0.19648442089349655 0.6870131543627426 2.7759090872853025
- link LeftLeg: geometry collision box size=2.8536410994455483 0.28526260733876685 0.21329385128670925; visual box size=2.8536410994455483 0.28526260733876685 0.21329385128670925
- link LeftLowerLeg: geometry collision box size=0.1 0.3947411167343772 0.1; visual box size=0.1 0.3947411167343772 0.1
- link RightLeg: geometry collision box size=1.8124778391001857 0.1 0.12409585248661345; visual box size=1.8124778391001857 0.1 0.12409585248661345
- link RightLowerLeg: geometry collision box size=0.7828771702108559 0.3624308573166486 2.450725652209476; visual box size=0.7828771702108559 0.3624308573166486 2.450725652209476
Joints:
- joint Torso_BackLowerLeg: origin xyz=0 -1.9867890771051135 0 rpy=0 0 0 -> xyz=0 -1.58913512194184 0 rpy=0 0 0
- joint Torso_FrontLowerLeg: origin xyz=0 1.783038989306366 0 rpy=0 0 0 -> xyz=0 1.0182689891632226 0 rpy=0 0 0
- joint Torso_LeftLowerLeg: origin xyz=-2.3484619884504316 0 0 rpy=0 0 0 -> xyz=-2.8536410994455483 0 0 rpy=0 0 0
- joint Torso_RightLowerLeg: origin xyz=1.9065036648992153 0 0 rpy=0 0 0 -> xyz=1.8124778391001857 0 0 rpy=0 0 0

File: body110.urdf (robot description, URDF)
Before this commit: robot robot, 9 links, 8 joints
Links:
- link BackLeg: geometry collision box size=0.13896963867027845 1.5693676591292212 0.17732307928056504; visual box size=0.13896963867027845 1.5693676591292212 0.17732307928056504
- link BackLowerLeg: geometry collision box size=0.6239230226133327 0.7775535398938561 2.6017967790972536; visual box size=0.6239230226133327 0.7775535398938561 2.6017967790972536
- link FrontLeg: geometry collision box size=0.8776895945553691 1.0055845613826715 0.1; visual box size=0.8776895945553691 1.0055845613826715 0.1
- link FrontLowerLeg: geometry collision box size=0.276589778756831 0.8243894910754616 2.443925938390503; visual box size=0.276589778756831 0.8243894910754616 2.443925938390503
- link LeftLeg: geometry collision box size=2.7884465453231844 0.1669207984402046 0.39327310865998466; visual box size=2.7884465453231844 0.1669207984402046 0.39327310865998466
- link LeftLowerLeg: geometry collision box size=0.1 0.3963902449449713 0.3044058872569002; visual box size=0.1 0.3963902449449713 0.3044058872569002
- link RightLeg: geometry collision box size=1.572104666333804 0.1858503699551585 0.3434364071295719; visual box size=1.572104666333804 0.1858503699551585 0.3434364071295719
- link RightLowerLeg: geometry collision box size=0.9014126149219928 0.2056636502648006 2.63797159961483; visual box size=0.9014126149219928 0.2056636502648006 2.63797159961483
Joints:
- joint Torso_BackLowerLeg: origin xyz=0 -1.7228012178574785 0 rpy=0 0 0 -> xyz=0 -1.5693676591292212 0 rpy=0 0 0
- joint Torso_FrontLowerLeg: origin xyz=0 2.261069071281585 0 rpy=0 0 0 -> xyz=0 1.0055845613826715 0 rpy=0 0 0
- joint Torso_LeftLowerLeg: origin xyz=-2.6666621890226283 0 0 rpy=0 0 0 -> xyz=-2.7884465453231844 0 0 rpy=0 0 0
- joint Torso_RightLowerLeg: origin xyz=1.8060509147898207 0 0 rpy=0 0 0 -> xyz=1.572104666333804 0 0 rpy=0 0 0
