Commit message: done

File: body111.urdf (robot description, URDF)
Before this commit: robot robot, 9 links, 8 joints
Links:
- link BackLeg: geometry collision box size=0.40184613413014586 1.7079013864047676 0.36536972340048457; visual box size=0.40184613413014586 1.7079013864047676 0.36536972340048457
- link BackLowerLeg: geometry collision box size=0.8204541531813919 0.8309023887028678 2.546466493364782; visual box size=0.8204541531813919 0.8309023887028678 2.546466493364782
- link FrontLeg: geometry collision box size=0.9225325262326058 0.8526377279066053 0.1; visual box size=0.9225325262326058 0.8526377279066053 0.1
- link FrontLowerLeg: geometry collision box size=0.1 0.5540404676573223 2.5028334411603397; visual box size=0.1 0.5540404676573223 2.5028334411603397
- link LeftLeg: geometry collision box size=2.7039010566087014 0.29903687205340734 0.3457748326895418; visual box size=2.7039010566087014 0.29903687205340734 0.3457748326895418
- link LeftLowerLeg: geometry collision box size=0.1 0.4284055321000022 0.1; visual box size=0.1 0.4284055321000022 0.1
- link RightLeg: geometry collision box size=1.805360755776599 0.1 0.27206311413047624; visual box size=1.805360755776599 0.1 0.27206311413047624
- link RightLowerLeg: geometry collision box size=0.902782676288756 0.10112023451757252 2.338244283890686; visual box size=0.902782676288756 0.10112023451757252 2.338244283890686
Joints:
- joint Torso_BackLowerLeg: origin xyz=0 -1.8362002236309234 0 rpy=0 0 0 -> xyz=0 -1.7079013864047676 0 rpy=0 0 0
- joint Torso_FrontLowerLeg: origin xyz=0 2.0183237727431362 0 rpy=0 0 0 -> xyz=0 0.8526377279066053 0 rpy=0 0 0
- joint Torso_LeftLowerLeg: origin xyz=-2.240413471567521 0 0 rpy=0 0 0 -> xyz=-2.7039010566087014 0 0 rpy=0 0 0
- joint Torso_RightLowerLeg: origin xyz=1.8656436791279858 0 0 rpy=0 0 0 -> xyz=1.805360755776599 0 0 rpy=0 0 0

File: body112.urdf (robot description, URDF)
Before this commit: robot robot, 9 links, 8 joints
Links:
- link BackLeg: geometry collision box size=0.3374347996024306 1.5072676362668924 0.1; visual box size=0.3374347996024306 1.5072676362668924 0.1
- link BackLowerLeg: geometry collision box size=0.9768834585177595 0.7297405749415289 2.3059975085253086; visual box size=0.9768834585177595 0.7297405749415289 2.3059975085253086
- link FrontLeg: geometry collision box size=0.8549740098762859 0.905509894365635 0.19560129294141312; visual box size=0.8549740098762859 0.905509894365635 0.19560129294141312
- link FrontLowerLeg: geometry collision box size=0.2263212805288094 0.6697729467705829 2.7471782258311492; visual box size=0.2263212805288094 0.6697729467705829 2.7471782258311492
- link LeftLeg: geometry collision box size=2.909129121260114 0.23143393726231848 0.4370777757524497; visual box size=2.909129121260114 0.23143393726231848 0.4370777757524497
- link LeftLowerLeg: geometry collision box size=0.1 0.6058107609249561 0.1; visual box size=0.1 0.6058107609249561 0.1
- link RightLeg: geometry collision box size=1.5535766230799648 0.15756287938135224 0.21441596525078746; visual box size=1.5535766230799648 0.15756287938135224 0.21441596525078746
- link RightLowerLeg: geometry collision box size=0.9387224235156142 0.1 2.3030831949664665; visual box size=0.9387224235156142 0.1 2.3030831949664665
Joints:
- joint Torso_BackLowerLeg: origin xyz=0 -1.8959922776560694 0 rpy=0 0 0 -> xyz=0 -1.5072676362668924 0 rpy=0 0 0
- joint Torso_FrontLowerLeg: origin xyz=0 2.1052136391747887 0 rpy=0 0 0 -> xyz=0 0.905509894365635 0 rpy=0 0 0
- joint Torso_LeftLowerLeg: origin xyz=-1.9508197224662465 0 0 rpy=0 0 0 -> xyz=-2.909129121260114 0 0 rpy=0 0 0
- joint Torso_RightLowerLeg: origin xyz=1.809461385025319 0 0 rpy=0 0 0 -> xyz=1.5535766230799648 0 0 rpy=0 0 0

File: body113.urdf (robot description, URDF)
Before this commit: robot robot, 9 links, 8 joints
Links:
- link BackLeg: geometry collision box size=0.4686312106851365 1.8161392734198574 0.1; visual box size=0.4686312106851365 1.8161392734198574 0.1
- link BackLowerLeg: geometry collision box size=0.7117766366306434 0.8200643294717855 2.547220236741532; visual box size=0.7117766366306434 0.8200643294717855 2.547220236741532
- link FrontLeg: geometry collision box size=1.043578256422464 1.110431453337141 0.1; visual box size=1.043578256422464 1.110431453337141 0.1
- link FrontLowerLeg: geometry collision box size=0.1657864759903068 0.7816986469557488 2.720547262036788; visual box size=0.1657864759903068 0.7816986469557488 2.720547262036788
- link LeftLeg: geometry collision box size=2.8402844378835006 0.2898041825691668 0.3328306497224124; visual box size=2.8402844378835006 0.2898041825691668 0.3328306497224124
- link LeftLowerLeg: geometry collision box size=0.1 0.4948258113520584 0.2330107686799552; visual box size=0.1 0.4948258113520584 0.2330107686799552
- link RightLeg: geometry collision box size=1.4896338882349358 0.21731420504957252 0.2305506273743668; visual box size=1.4896338882349358 0.21731420504957252 0.2305506273743668
- link RightLowerLeg: geometry collision box size=0.8278432871724988 0.1660227431644451 2.6359191896295706; visual box size=0.8278432871724988 0.1660227431644451 2.6359191896295706
Joints:
- joint Torso_BackLowerLeg: origin xyz=0 -1.8113602057350926 0 rpy=0 0 0 -> xyz=0 -1.8161392734198574 0 rpy=0 0 0
- joint Torso_FrontLowerLeg: origin xyz=0 2.1821356455321004 0 rpy=0 0 0 -> xyz=0 1.110431453337141 0 rpy=0 0 0
- joint Torso_LeftLowerLeg: origin xyz=-2.1139107156794403 0 0 rpy=0 0 0 -> xyz=-2.8402844378835006 0 0 rpy=0 0 0
- joint Torso_RightLowerLeg: origin xyz=2.204686634784818 0 0 rpy=0 0 0 -> xyz=1.4896338882349358 0 0 rpy=0 0 0

File: body114.urdf (robot description, URDF)
Before this commit: robot robot, 9 links, 8 joints
Links:
- link BackLeg: geometry collision box size=0.16770689713221298 1.6778388245194562 0.1; visual box size=0.16770689713221298 1.6778388245194562 0.1
- link BackLowerLeg: geometry collision box size=0.6581167390428214 0.8659966687943037 2.514598481244127; visual box size=0.6581167390428214 0.8659966687943037 2.514598481244127
- link FrontLeg: geometry collision box size=0.8792664021719978 0.8497495594082592 0.2567031053944545; visual box size=0.8792664021719978 0.8497495594082592 0.2567031053944545
- link FrontLowerLeg: geometry collision box size=0.1434259083120863 0.5988501072293495 2.7508361451897514; visual box size=0.1434259083120863 0.5988501072293495 2.7508361451897514
- link LeftLeg: geometry collision box size=2.8687355483594428 0.13847849793533784 0.1082402037898007; visual box size=2.8687355483594428 0.13847849793533784 0.1082402037898007
- link LeftLowerLeg: geometry collision box size=0.1 0.5355670304453641 0.21284942506389495; visual box size=0.1 0.5355670304453641 0.21284942506389495
- link RightLeg: geometry collision box size=1.8456766531850382 0.19299633929437346 0.1; visual box size=1.8456766531850382 0.19299633929437346 0.1
- link RightLowerLeg: geometry collision box size=0.6023569617435398 0.45724880606318075 2.6735715086375973; visual box size=0.6023569617435398 0.45724880606318075 2.6735715086375973
Joints:
- joint Torso_BackLowerLeg: origin xyz=0 -1.8107235754557456 0 rpy=0 0 0 -> xyz=0 -1.6778388245194562 0 rpy=0 0 0
- joint Torso_FrontLowerLeg: origin xyz=0 1.8941254871252515 0 rpy=0 0 0 -> xyz=0 0.8497495594082592 0 rpy=0 0 0
- joint Torso_LeftLowerLeg: origin xyz=-2.032198119503865 0 0 rpy=0 0 0 -> xyz=-2.8687355483594428 0 0 rpy=0 0 0
- joint Torso_RightLowerLeg: origin xyz=1.8211409946917998 0 0 rpy=0 0 0 -> xyz=1.8456766531850382 0 0 rpy=0 0 0

File: body115.urdf (robot description, URDF)
Before this commit: robot robot, 9 links, 8 joints
Links:
- link BackLeg: geometry collision box size=0.10645497517310201 1.5471132029372499 0.3756592833632322; visual box size=0.10645497517310201 1.5471132029372499 0.3756592833632322
- link BackLowerLeg: geometry collision box size=0.601421988755277 0.7032272906768198 2.518435392426231; visual box size=0.601421988755277 0.7032272906768198 2.518435392426231
- link FrontLeg: geometry collision box size=0.9150800320417048 1.1727348210361945 0.1; visual box size=0.9150800320417048 1.1727348210361945 0.1
- link FrontLowerLeg: geometry collision box size=0.313554958451554 0.7223703664922889 2.6329263853403018; visual box size=0.313554958451554 0.7223703664922889 2.6329263853403018
- link LeftLeg: geometry collision box size=2.945871345638401 0.42162011762059876 0.3547607641807942; visual box size=2.945871345638401 0.42162011762059876 0.3547607641807942
- link LeftLowerLeg: geometry collision box size=0.16019601527807212 0.40583765574743247 0.16749468813992122; visual box size=0.16019601527807212 0.40583765574743247 0.16749468813992122
- link RightLeg: geometry collision box size=1.8513165993388343 0.17857194125282863 0.13669290182920613; visual box size=1.8513165993388343 0.17857194125282863 0.13669290182920613
- link RightLowerLeg: geometry collision box size=0.9774743848912057 0.22293583212688248 2.4780657974540263; visual box size=0.9774743848912057 0.22293583212688248 2.4780657974540263
Joints:
- joint Torso_BackLowerLeg: origin xyz=0 -2.0198047188459354 0 rpy=0 0 0 -> xyz=0 -1.5471132029372499 0 rpy=0 0 0
- joint Torso_FrontLowerLeg: origin xyz=0 1.9418716320336495 0 rpy=0 0 0 -> xyz=0 1.1727348210361945 0 rpy=0 0 0
- joint Torso_LeftLowerLeg: origin xyz=-1.807862083749035 0 0 rpy=0 0 0 -> xyz=-2.945871345638401 0 0 rpy=0 0 0
- joint Torso_RightLowerLeg: origin xyz=1.8816543916579573 0 0 rpy=0 0 0 -> xyz=1.8513165993388343 0 0 rpy=0 0 0

File: body116.urdf (robot description, URDF)
Before this commit: robot robot, 9 links, 8 joints
Links:
- link BackLeg: geometry collision box size=0.1164107373377585 1.4384320303482188 0.28220342661530207; visual box size=0.1164107373377585 1.4384320303482188 0.28220342661530207
- link BackLowerLeg: geometry collision box size=0.8620251214755804 0.7770143593857235 2.622769094250817; visual box size=0.8620251214755804 0.7770143593857235 2.622769094250817
- link FrontLeg: geometry collision box size=0.897348714391234 0.9838876528899343 0.3468051303655457; visual box size=0.897348714391234 0.9838876528899343 0.3468051303655457
- link FrontLowerLeg: geometry collision box size=0.2595221367228875 0.7816578694266869 2.6796386480707852; visual box size=0.2595221367228875 0.7816578694266869 2.6796386480707852
- link LeftLeg: geometry collision box size=2.5654183943908295 0.4596701066947707 0.12100925540855756; visual box size=2.5654183943908295 0.4596701066947707 0.12100925540855756
- link LeftLowerLeg: geometry collision box size=0.11563071332954103 0.5633020376334266 0.1; visual box size=0.11563071332954103 0.5633020376334266 0.1
- link RightLeg: geometry collision box size=1.5807978469432875 0.29575797441334173 0.17619019405960562; visual box size=1.5807978469432875 0.29575797441334173 0.17619019405960562
- link RightLowerLeg: geometry collision box size=0.8116729537762423 0.4131456057324274 2.6382619686433406; visual box size=0.8116729537762423 0.4131456057324274 2.6382619686433406
Joints:
- joint Torso_BackLowerLeg: origin xyz=0 -2.100894773744707 0 rpy=0 0 0 -> xyz=0 -1.4384320303482188 0 rpy=0 0 0
- joint Torso_FrontLowerLeg: origin xyz=0 1.6990438456463894 0 rpy=0 0 0 -> xyz=0 0.9838876528899343 0 rpy=0 0 0
- joint Torso_LeftLowerLeg: origin xyz=-1.9182091093276734 0 0 rpy=0 0 0 -> xyz=-2.5654183943908295 0 0 rpy=0 0 0
- joint Torso_RightLowerLeg: origin xyz=2.1617375575810893 0 0 rpy=0 0 0 -> xyz=1.5807978469432875 0 0 rpy=0 0 0

File: body117.urdf (robot description, URDF)
Before this commit: robot robot, 9 links, 8 joints
Links:
- link BackLeg: geometry collision box size=0.33560648273412813 1.5482946754334832 0.34953290761892974; visual box size=0.33560648273412813 1.5482946754334832 0.34953290761892974
- link BackLowerLeg: geometry collision box size=0.8976858833306738 0.8415736087136374 2.5727287184423937; visual box size=0.8976858833306738 0.8415736087136374 2.5727287184423937
- link FrontLeg: geometry collision box size=0.9325547472955973 1.1684896666139726 0.2728387722595213; visual box size=0.9325547472955973 1.1684896666139726 0.2728387722595213
- link FrontLowerLeg: geometry collision box size=0.1 0.46971881494660406 2.7690927278813335; visual box size=0.1 0.46971881494660406 2.7690927278813335
- link LeftLeg: geometry collision box size=2.844798078566333 0.39223053774180244 0.37676763643576416; visual box size=2.844798078566333 0.39223053774180244 0.37676763643576416
- link LeftLowerLeg: geometry collision box size=0.11958211556152501 0.4708725967462052 0.2377644890453163; visual box size=0.11958211556152501 0.4708725967462052 0.2377644890453163
- link RightLeg: geometry collision box size=1.6143320291750778 0.15730848992191857 0.3827984351287472; visual box size=1.6143320291750778 0.15730848992191857 0.3827984351287472
- link RightLowerLeg: geometry collision box size=0.6574410629688863 0.2061611320816345 2.39106991039491; visual box size=0.6574410629688863 0.2061611320816345 2.39106991039491
Joints:
- joint Torso_BackLowerLeg: origin xyz=0 -1.7421605694104603 0 rpy=0 0 0 -> xyz=0 -1.5482946754334832 0 rpy=0 0 0
- joint Torso_FrontLowerLeg: origin xyz=0 1.886829465938331 0 rpy=0 0 0 -> xyz=0 1.1684896666139726 0 rpy=0 0 0
- joint Torso_LeftLowerLeg: origin xyz=-2.3016006988245654 0 0 rpy=0 0 0 -> xyz=-2.844798078566333 0 0 rpy=0 0 0
- joint Torso_RightLowerLeg: origin xyz=2.0336533121527336 0 0 rpy=0 0 0 -> xyz=1.6143320291750778 0 0 rpy=0 0 0

File: body118.urdf (robot description, URDF)
Before this commit: robot robot, 9 links, 8 joints
Links:
- link BackLeg: geometry collision box size=0.1031496396314342 1.5587283033923551 0.1; visual box size=0.1031496396314342 1.5587283033923551 0.1
- link BackLowerLeg: geometry collision box size=0.6512564866771082 0.6612144760382637 2.2854450430484134; visual box size=0.6512564866771082 0.6612144760382637 2.2854450430484134
- link FrontLeg: geometry collision box size=0.9479325220597548 1.110173852413272 0.33562488357314446; visual box size=0.9479325220597548 1.110173852413272 0.33562488357314446
- link FrontLowerLeg: geometry collision box size=0.1 0.698301712136842 2.7348068799417904; visual box size=0.1 0.698301712136842 2.7348068799417904
- link LeftLeg: geometry collision box size=2.646062295974912 0.37172846848530816 0.3560584201634628; visual box size=2.646062295974912 0.37172846848530816 0.3560584201634628
- link LeftLowerLeg: geometry collision box size=0.1 0.4858948129376166 0.3021982460580943; visual box size=0.1 0.4858948129376166 0.3021982460580943
- link RightLeg: geometry collision box size=1.8201017429764046 0.1 0.29976794151680325; visual box size=1.8201017429764046 0.1 0.29976794151680325
- link RightLowerLeg: geometry collision box size=0.796920255897801 0.31125015525755445 2.640904514882129; visual box size=0.796920255897801 0.31125015525755445 2.640904514882129
Joints:
- joint Torso_BackLowerLeg: origin xyz=0 -2.2452163451653515 0 rpy=0 0 0 -> xyz=0 -1.5587283033923551 0 rpy=0 0 0
- joint Torso_FrontLowerLeg: origin xyz=0 2.4549858672195097 0 rpy=0 0 0 -> xyz=0 1.110173852413272 0 rpy=0 0 0
- joint Torso_LeftLowerLeg: origin xyz=-2.165560383749802 0 0 rpy=0 0 0 -> xyz=-2.646062295974912 0 0 rpy=0 0 0
- joint Torso_RightLowerLeg: origin xyz=1.9314930525344909 0 0 rpy=0 0 0 -> xyz=1.8201017429764046 0 0 rpy=0 0 0
